File: front_wheels.kicad_sch (KiCad schematic)
At the start: 5 parts, among them M3 Motor_DC, M4 Motor_DC, U3 TB6612FNG

Commit message: some updates
Parts:
- removed C11, C12: 0.1uF, Capacitor_SMD:C_0805_2012Metric, symbol Device:C
- added C14, C7: 0.1uF, Capacitor_SMD:C_0805_2012Metric, symbol Device:C
- added C8: 10uF, Capacitor_Tantalum_SMD:CP_EIA-3216-18_Kemet-A, symbol Device:C_Polarized
Connections:
- net +3V3: now also C14.1
- net +5V: now also C7.1, C8.1
- net GND: now also C14.2, C7.2, C8.2
