File: rear_wheels.kicad_sch (KiCad schematic)
At the start: 5 parts, among them M5 Motor_DC, M6 Motor_DC, U8 TB6612FNG

Commit message: some updates
Parts:
- removed C14: 0.1uF, Capacitor_SMD:C_0805_2012Metric, symbol Device:C
- added C1: 10uF, Capacitor_Tantalum_SMD:CP_EIA-3216-18_Kemet-A, symbol Device:C_Polarized
- added C3: 0.1uF, Capacitor_SMD:C_0805_2012Metric, symbol Device:C
Connections:
- net +3V3: now also C3.1
- net +5V: now also C1.1
- net GND: now also C1.2, C3.2
