File: rover-circuit.kicad_pcb (KiCad board)
At the start: 2 copper layers, 343.2 x 98.5 mm, 52 parts, among them J1 Battery, J2 USB_C_Receptacle_USB2.0_14P, J3 Recharge Connector, J4 Display Connector, J5 Raspberry_Pi_2_3, M3 Motor_DC, M4 Motor_DC, M5 Motor_DC, M6 Motor_DC, Q1 AO3401A, SW1 SW_EN, SW2 SW_IO0, SW3 SW_SPDT, U1 LM3671MFX-1.25_NOPB, U2 ESP32-S3-WROOM-1, U3 TB6612FNG, U4 LM2596S-5, U7 INA219AxD, U8 TB6612FNG

Commit message: some updates
Parts:
- removed D1, D5: SS34, Diode_SMD:D_SMA
- removed J3: Recharge Connector, Connector_JST:JST_EH_B2B-EH-A_1x02_P2.50mm_Vertical
- removed L1: 33uH, Inductor_SMD:L_10.4x10.4_H4.8
- removed L2: 22uH, Inductor_SMD:L_Taiyo-Yuden_MD-5050
- removed Q1: AO3401A, Package_TO_SOT_SMD:SOT-23
- removed R2: 100K, Resistor_SMD:R_0805_2012Metric
- removed SW3: SW_SPDT, Button_Switch_THT:SW_Slide_SPDT_Angled_CK_OS102011MA1Q
- removed U4: LM2596S-5, Package_TO_SOT_SMD:TO-263-5_TabPin3
- removed U7: INA219AxD, Package_SO:SOIC-8_3.9x4.9mm_P1.27mm
- added C10: 10uF, Capacitor_SMD:C_0603_1608Metric, F.Cu at (143.8, 130.2)
- added C13: 10uF, Capacitor_SMD:C_0603_1608Metric, F.Cu at (142.0, 130.2)
- added C15: 10uF, Capacitor_SMD:C_0603_1608Metric, F.Cu at (141.6, 118.4)
- added C16: 10uF, Capacitor_SMD:C_0603_1608Metric, F.Cu at (143.4, 118.4)
- added C17: 10uF, Capacitor_SMD:C_0603_1608Metric, F.Cu at (134.8, 118.4)
- added C18: 0.1uF, Capacitor_SMD:C_0402_1005Metric, F.Cu at (138.7, 122.4)
- added C19: 1uF, Capacitor_SMD:C_0805_2012Metric, F.Cu at (122.0, 126.2)
- added C2: 10uF, Capacitor_SMD:C_0603_1608Metric, F.Cu at (135.2, 130.2)
- added C20: 4.7uF, Capacitor_SMD:C_0805_2012Metric, F.Cu at (118.6, 131.6)
- added C21: 4.7uF, Capacitor_SMD:C_0805_2012Metric, F.Cu at (126.3, 131.8)
- added C22: 0.1uF, Capacitor_SMD:C_0805_2012Metric, F.Cu at (118.0, 122.0)
- added C23: 22uF, Capacitor_SMD:C_1210_3225Metric, F.Cu at (115.0, 121.4)
- added C24: 10nF, Capacitor_SMD:C_0805_2012Metric, F.Cu at (-117.8, 153.5)
- added C25: 0.1uF, Capacitor_SMD:C_0805_2012Metric, F.Cu at (124.4, 119.2)
- added C9: 0.1uF, Capacitor_SMD:C_0402_1005Metric, F.Cu at (139.1, 134.2)
- added D3: GREEN, LED_SMD:LED_0402_1005Metric, F.Cu at (117.2, 134.9)
- added D4: YELLOW, LED_SMD:LED_0402_1005Metric, F.Cu at (117.2, 136.5)
- added JP4: Battery Jumper, Jumper:SolderJumper-2_P1.3mm_Bridged2Bar_RoundedPad1.0x1.5mm, F.Cu at (129.1, 130.8)
- added L3: 2.2uH, Inductor_SMD:L_Coilcraft_LPS3010, F.Cu at (138.6, 126.6)
- added L4: 2.2uH, Inductor_SMD:L_Coilcraft_LPS3010, F.Cu at (138.2, 114.8)
- added MT1: ICM-42670-P, ICM-42670-P:XDCR_ICM-42670-P, F.Cu at (-90.5, 156.0)
- added R4: 100, Resistor_SMD:R_0402_1005Metric, F.Cu at (136.8, 134.2)
- added R5: 100, Resistor_SMD:R_0402_1005Metric, F.Cu at (136.5, 122.4)
- added R7: 1.5K, Resistor_SMD:R_0402_1005Metric, F.Cu at (115.1, 134.9)
- added R8: 1.5K, Resistor_SMD:R_0402_1005Metric, F.Cu at (115.1, 136.5)
- added R9: 10K, Resistor_SMD:R_0402_1005Metric, F.Cu at (118.9, 129.2)
- added SW4: SW_SPDT, Button_Switch_THT:SW_Slide_SPDT_Angled_CK_OS102011MA1Q, F.Cu at (173.6, 134.8)
- added TP1: Batt Out, TestPoint:TestPoint_Pad_D1.0mm, F.Cu at (-189.5, 127.8)
- added TP2: Batt, TestPoint:TestPoint_Pad_D1.0mm, F.Cu at (-189.5, 131.4)
- added TP3: SDA, TestPoint:TestPoint_Pad_D1.0mm, F.Cu at (-186.2, 128.0)
- added TP4: SCL, TestPoint:TestPoint_Pad_D1.0mm, F.Cu at (-186.2, 131.1)
- added U5: BQ24074RGT, Package_DFN_QFN:VQFN-16-1EP_3x3mm_P0.5mm_EP1.6x1.6mm, F.Cu at (122.2, 130.8)
- added U6: TPS63001, Package_SON:Texas_DRC0010J_ThermalVias, F.Cu at (138.6, 131.0)
- added U9: TPS63002, Package_SON:Texas_DRC0010J_ThermalVias, F.Cu at (138.2, 119.2)
- C1, C8: footprint Capacitor_SMD:C_0805_2012Metric -> Capacitor_Tantalum_SMD:CP_EIA-3216-18_Kemet-A
- C11: value 0.1uF -> 2.2uF
- C3: value 220uF -> 0.1uF; footprint Capacitor_SMD:CP_Elec_6.3x7.7 -> Capacitor_SMD:C_0805_2012Metric
- C7: value 680uF -> 0.1uF; footprint Capacitor_SMD:CP_Elec_10x10 -> Capacitor_SMD:C_0805_2012Metric
- J1: value Battery -> 1S2P 18650 Pack
- R10: value 4.7K -> 1.13K; footprint Resistor_SMD:R_0805_2012Metric -> Resistor_SMD:R_0402_1005Metric
- R11: value 4.7K -> 1.18K; footprint Resistor_SMD:R_0805_2012Metric -> Resistor_SMD:R_0402_1005Metric
- R3: value 0 -> 4.12K; footprint Resistor_SMD:R_0805_2012Metric -> Resistor_SMD:R_0402_1005Metric
- U1: value LM3671MFX-1.25_NOPB -> INA219AxDCN; footprint Package_TO_SOT_SMD:SOT-23-5 -> Package_TO_SOT_SMD:SOT-23-8
- moved C3 250.9 mm to (122.0, 101.0)
- moved U1 232.1 mm to (124.2, 122.2), turned to 180 degrees
- moved C1 229.7 mm to (121.2, 114.4), turned to 180 degrees
- moved R1 225.9 mm to (129.7, 122.8), turned to -90 degrees
- moved R11 216.0 mm to (124.9, 128.5)
- moved R10 212.0 mm to (118.9, 128.1), turned to 180 degrees
- moved J1 206.0 mm to (110.8, 122.8), turned to 90 degrees
- moved R3 194.7 mm to (118.9, 127.0), turned to 180 degrees
- moved U8 191.8 mm to (119.0, 106.6), turned to 0 degrees
- moved M6 190.7 mm to (110.8, 112.2), turned to 90 degrees
- moved C4 186.6 mm to (121.7, 112.2), turned to 180 degrees
- moved M5 180.7 mm to (110.8, 103.4), turned to 90 degrees
- moved M4 169.3 mm to (110.8, 93.7), turned to 90 degrees
- moved M3 160.1 mm to (110.8, 84.8), turned to 90 degrees
- moved C14 152.5 mm to (-207.4, 159.7), turned to 0 degrees
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Connections:
- C1 pad 1: Net-(D1-K) -> +5V
- C11 pad 1: +5V -> +3V3
- C12 pad 1: +5V -> GND
- C12 pad 2: GND -> +3V3
- C14 pad 1: +5V -> +3V3
- C3 pad 1: +5V -> +3V3
- C7 pad 1: VBATT -> +5V
- C8 pad 1: +3V3 -> +5V
- J1 pad 1: /IN+ -> /Battery Circuit/BAT
- J2 pad S1: Net-(J2-SHIELD) -> GND
- J5 pad 1: Net-(J5-3V3-Pad1) -> unconnected-(J5-3V3-Pad1)_1
- J5 pad 10: unconnected-(J5-GPIO15/RXD-Pad10) -> /TX
- J5 pad 11: unconnected-(J5-GPIO17-Pad11) -> /BIN1_1
- J5 pad 12: unconnected-(J5-GPIO18/PWM0-Pad12) -> /PWMA_1
- J5 pad 13: unconnected-(J5-GPIO27-Pad13) -> /AIN2_2
- J5 pad 14: Net-(J5-GND-Pad14) -> GND
- J5 pad 15: unconnected-(J5-GPIO22-Pad15) -> /BIN2_1
- J5 pad 16: unconnected-(J5-GPIO23-Pad16) -> /STBYA
- J5 pad 17: Net-(J5-3V3-Pad1) -> unconnected-(J5-3V3-Pad1)
- J5 pad 18: unconnected-(J5-GPIO24-Pad18) -> /BIN1_2
- J5 pad 2: Net-(J5-5V-Pad2) -> +5V
- J5 pad 20: Net-(J5-GND-Pad14) -> GND
- J5 pad 21: unconnected-(J5-MISO0/GPIO9-Pad21) -> /MISO
- J5 pad 22: unconnected-(J5-GPIO25-Pad22) -> /BIN2_2
- J5 pad 23: unconnected-(J5-SCLK0/GPIO11-Pad23) -> /CLK
- J5 pad 25: Net-(J5-GND-Pad14) -> GND
- J5 pad 3: unconnected-(J5-SDA/GPIO2-Pad3) -> /SDA
- J5 pad 30: Net-(J5-GND-Pad14) -> GND
- J5 pad 32: unconnected-(J5-PWM0/GPIO12-Pad32) -> /PWMB_2
- J5 pad 33: unconnected-(J5-PWM1/GPIO13-Pad33) -> /PWMA_2
- J5 pad 34: Net-(J5-GND-Pad14) -> GND
- J5 pad 35: unconnected-(J5-GPIO19/MISO1-Pad35) -> /PWMB_1
- J5 pad 36: unconnected-(J5-GPIO16-Pad36) -> /STBYB
- J5 pad 37: unconnected-(J5-GPIO26-Pad37) -> /AIN1_2
- J5 pad 38: unconnected-(J5-GPIO20/MOSI1-Pad38) -> /AIN1_1
- J5 pad 39: Net-(J5-GND-Pad14) -> GND
- J5 pad 4: Net-(J5-5V-Pad2) -> +5V
- J5 pad 40: unconnected-(J5-GPIO21/SCLK1-Pad40) -> /AIN2_1
- J5 pad 5: unconnected-(J5-SCL/GPIO3-Pad5) -> /SCL
- J5 pad 6: Net-(J5-GND-Pad14) -> GND
- J5 pad 8: unconnected-(J5-GPIO14/TXD-Pad8) -> /RX
- J5 pad 9: Net-(J5-GND-Pad14) -> GND
- R1 pad 2: /IN+ -> /Battery Circuit/IN+
- R10 pad 1: +3V3 -> Net-(U5-ISET)
- R10 pad 2: /SDA -> GND
- R11 pad 1: +3V3 -> Net-(U5-ILIM)
- R11 pad 2: /SCL -> GND
- R3 pad 1: Net-(J2-SHIELD) -> Net-(U5-ITERM)
- U1 pad 1: Net-(D1-K) -> /Battery Circuit/IN+
- U1 pad 2: GND -> VBATT
- U1 pad 3: Net-(D1-K) -> GND
- U1 pad 5: Net-(U1-SW) -> /SCL
- U2 pad 36: unconnected-(U2-RXD0-Pad36) -> /RX
- U2 pad 37: unconnected-(U2-TXD0-Pad37) -> /TX
Routing:
- net (no net): track 0.00 -> 213.1 mm, vias 0 -> 5
- net Net-(SW3-B): track 94.8 -> 0.00 mm, vias 2 -> 0
- net Net-(D1-K): track 53.1 -> 0.00 mm, vias 2 -> 0
- net /IN+: track 21.4 -> 0.00 mm
- net Net-(J2-SHIELD): track 20.5 -> 0.00 mm, vias 1 -> 0
- net Net-(D5-K): track 19.4 -> 0.00 mm
- net VBATT: track 75.3 -> 93.1 mm, vias 2 -> 6
- net /Battery Circuit/BATT_OUT: track 0.00 -> 15.6 mm, vias 0 -> 2
- net GND: track 41.4 -> 53.4 mm, vias 32 -> 49
- net /Battery Circuit/BAT: track 0.00 -> 10.7 mm
- net Net-(D4-K): track 0.00 -> 10.1 mm
- net +3V3: track 205.6 -> 214.9 mm, vias 5 -> 7
- net Net-(D3-K): track 0.00 -> 6.79 mm
- net Net-(M5-+): track 7.73 -> 13.7 mm
- net Net-(M5--): track 7.69 -> 13.6 mm
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- added copper zone on F.Cu, net +3V3
- added copper zone on F.Cu, net +5V
- added copper zone on F.Cu, net /Battery Circuit/BAT
- added copper zone on F.Cu, net /Battery Circuit/BATT_OUT
- added copper zone on F.Cu, net Net-(M5-+)
- added copper zone on F.Cu, net Net-(M5--)
- added copper zone on F.Cu, net Net-(M6-+)
- added copper zone on F.Cu, net Net-(M6--)
- added copper zone on F.Cu, net Net-(U6-L1)
- added copper zone on F.Cu, net Net-(U6-L2)
- added copper zone on F.Cu, net Net-(U9-L1)
- added copper zone on F.Cu, net Net-(U9-L2)
- added copper zone on F.Cu, net VBATT

Commit message: add uwb module
Parts:
- added C26: 0.1uF, Capacitor_SMD:C_0805_2012Metric, F.Cu at (122.7, 150.8)
- added DWM1: DWM1000, RF_Module:DWM1000, F.Cu at (190.6, 125.2)
- added R15: 10K, Resistor_SMD:R_0402_1005Metric, F.Cu at (121.9, 153.3)
- added REF**: KiCad-Logo2_5mm_SilkScreen, Symbol:KiCad-Logo2_5mm_SilkScreen, F.Cu at (128.9, 72.6)
- added REF**: OSHW-Logo2_7.3x6mm_SilkScreen, Symbol:OSHW-Logo2_7.3x6mm_SilkScreen, F.Cu at (117.5, 72.8)
- moved C14 338.5 mm to (122.2, 82.4), turned to 180 degrees
- moved C7 335.2 mm to (121.8, 93.6), turned to 180 degrees
- moved C8 333.2 mm to (121.4, 95.8), turned to 180 degrees
- moved U3 269.9 mm to (119.1, 88.0)
- moved J4 1.20 mm to (205.2, 114.5)
Connections:
- J5 pad 19: unconnected-(J5-MOSI0/GPIO10-Pad19) -> /MOSI
- J5 pad 24: unconnected-(J5-~{CE0}/GPIO8-Pad24) -> /UWB_~{CS}
- U2 pad 15: /RES -> /UWB_IRQ
- U2 pad 16: /DC -> /CLK
- U2 pad 17: /CLK -> /MISO
- U2 pad 18: /MISO -> /MOSI
- U2 pad 19: /CS -> /UWB_~{CS}
- U2 pad 20: /STBYA -> /UWB_WU
- U2 pad 21: /PWMA_2 -> /UWB_~{RST}
- U2 pad 31: /SCL -> unconnected-(U2-IO38-Pad31)
- U2 pad 32: /SDA -> unconnected-(U2-IO39-Pad32)
- U2 pad 34: unconnected-(U2-IO41-Pad34) -> /SDA
- U2 pad 35: unconnected-(U2-IO42-Pad35) -> /SCL
Routing:
- net /RX: track 0.00 -> 62.4 mm
- net /TX: track 0.00 -> 62.4 mm
- net /SCL: track 89.9 -> 147.8 mm
- net /SDA: track 89.2 -> 147.1 mm
- net /CLK: track 110.6 -> 153.2 mm, vias 2 -> 4
- net /MISO: track 110.5 -> 152.6 mm, vias 2 -> 4
- net /UWB_WU: track 0.00 -> 35.4 mm, vias 0 -> 2
- net /UWB_~{RST}: track 0.00 -> 35.3 mm, vias 0 -> 2
- net /UWB_IRQ: track 0.00 -> 19.6 mm, vias 0 -> 1
- net /MOSI: track 0.00 -> 18.8 mm, vias 0 -> 1
- net /UWB_~{CS}: track 0.00 -> 18.8 mm, vias 0 -> 1
- net GND: vias 49 -> 52

Commit message: minors
Parts:
- added JP2: Disable ESP, TestPoint:TestPoint_Bridge_Pitch2.54mm_Drill0.7mm, F.Cu at (-39.3, 144.3)
- added R2: 4.7K, Resistor_SMD:R_0402_1005Metric, F.Cu at (-39.6, 147.0)
- added R6: 4.7K, Resistor_SMD:R_0402_1005Metric, F.Cu at (-39.6, 149.0)
Routing:
- net /SDA: track 147.1 -> 195.9 mm, vias 2 -> 4
- net /SCL: track 147.8 -> 193.8 mm, vias 2 -> 4
