File: rover-circuit.kicad_pcb (KiCad board)
At the start: 4 copper layers, 87 x 69.9 mm, 25 parts, among them J2 USB_C_Receptacle_USB2.0_14P, J5 Raspberry_Pi_2_3, J6 Conn_02x07_Odd_Even, SW1 SW_EN, SW2 SW_IO0, U1 ESP32-C6-MINI-1, U2 BQ25887RGE, U3 DRV8833PWP, U4 TPD2EUSB30, U6 MPU-6050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

Commit message: design pcb and place components
Parts:
- added C1: 100n, Capacitor_SMD:C_0402_1005Metric, F.Cu at (173.9, 128.0)
- added C17: 22uF, Capacitor_SMD:C_0805_2012Metric, F.Cu at (191.2, 129.5)
- added C18: 10uF, Capacitor_SMD:C_0805_2012Metric, F.Cu at (191.2, 132.5)
- added C26: 1uF, Capacitor_SMD:C_0402_1005Metric, F.Cu at (190.4, 135.0)
- added D3: LED, LED_SMD:LED_0603_1608Metric, F.Cu at (193.3, 126.2)
- added L2: 2.2uH, Inductor_SMD:L_APV_ANR3012, F.Cu at (195.7, 130.3)
- added R15: 100K, Resistor_SMD:R_0603_1608Metric, F.Cu at (195.4, 133.8)
- R13, R14: footprint Resistor_SMD:R_0805_2012Metric -> Resistor_SMD:R_0402_1005Metric
- moved H8 213.4 mm to (128.2, 104.4)
- moved U4 213.1 mm to (157.6, 122.4)
- moved R14 211.1 mm to (155.9, 122.2), turned to 90 degrees
- moved H2 209.4 mm to (124.3, 98.0)
- moved R13 208.0 mm to (158.9, 122.2), turned to 90 degrees
- moved H7 155.2 mm to (186.2, 104.4)
- moved H1 143.2 mm to (190.1, 98.0)
- moved J6 34.1 mm to (310.5, 109.1), turned to 90 degrees
- moved U7 25.9 mm to (311.7, 114.4)
- moved DWM1 20.5 mm to (128.5, 78.0)
- moved U1 7.54 mm to (187.6, 81.9)
- moved J5 1.56 mm to (157.2, 104.6)
- turned U8 to 90 degrees
Other:
- board size 87 x 69.9 mm -> 78 x 56.6 mm

Commit message: moving on routing
Parts:
- removed D4: B340, Diode_SMD:D_SMC
- removed H3, H4: MountingHole, MountingHole:MountingHole_3.2mm_M3_Pad
- removed H5, H6: MountingHole, MountingHole:MountingHole_2.5mm
- removed U8: TPS5430DDA, Package_SO:TI_SO-PowerPAD-8_ThermalVias
- added C12: 22uF, Capacitor_SMD:C_1206_3216Metric, F.Cu at (134.0, 96.5)
- added C13: 100nF, Capacitor_SMD:C_0603_1608Metric, F.Cu at (142.0, 92.6)
- added C19: 100nF, Capacitor_SMD:C_0603_1608Metric, F.Cu at (136.2, 110.2)
- added C2: 1uF, Capacitor_SMD:C_0603_1608Metric, F.Cu at (136.9, 86.7)
- added C20: 22uF, Capacitor_SMD:C_0805_2012Metric, F.Cu at (141.4, 116.9)
- added C21: 22uF, Capacitor_SMD:C_0805_2012Metric, F.Cu at (141.4, 119.0)
- added C22: 10uF, Capacitor_SMD:C_0805_2012Metric, F.Cu at (137.9, 116.9)
- added C23: 22uF, Capacitor_SMD:C_0805_2012Metric, F.Cu at (147.8, 94.8)
- added C24: 22uF, Capacitor_SMD:C_0805_2012Metric, F.Cu at (145.7, 94.8)
- added C25: 10uF, Capacitor_SMD:C_0805_2012Metric, F.Cu at (146.4, 98.1)
- added C28: 22uF, Capacitor_SMD:C_0805_2012Metric, F.Cu at (156.0, 94.8)
- added C3: 22uF, Capacitor_SMD:C_1206_3216Metric, F.Cu at (134.0, 94.1)
- added C4: 47nF, Capacitor_SMD:C_0603_1608Metric, F.Cu at (133.9, 91.6)
- added C5: 10uF, Capacitor_SMD:C_1206_3216Metric, F.Cu at (136.6, 89.8)
- added C6: 4.7uF, Capacitor_SMD:C_0603_1608Metric, F.Cu at (127.2, 91.3)
- added C7: 10uF, Capacitor_SMD:C_0805_2012Metric, F.Cu at (129.8, 91.8)
- added D1: RED, LED_SMD:LED_0603_1608Metric, F.Cu at (101.9, 90.0)
- added D2: GRN, LED_SMD:LED_0603_1608Metric, F.Cu at (101.9, 88.1)
- added J1: Battery Connector, Connector_JST:JST_PH_S4B-PH-K_1x04_P2.00mm_Horizontal, F.Cu at (130.9, 79.3)
- added L1: 1uH, Inductor_SMD:L_1008_2520Metric, F.Cu at (139.2, 89.5)
- added L3: 4.7uH, Inductor_SMD:L_Sunlord_MWSA0503S, F.Cu at (140.7, 112.9)
- added L4: 10uH, Inductor_SMD:L_Sunlord_MWSA0503S, F.Cu at (146.0, 90.0)
- added R1: 2.2k, Resistor_SMD:R_0603_1608Metric, F.Cu at (105.0, 90.0)
- added R11: 64.9k, Resistor_SMD:R_0603_1608Metric, F.Cu at (138.5, 96.6)
- added R12: 10k, Resistor_SMD:R_0603_1608Metric, F.Cu at (140.1, 96.6)
- added R2: 1.1K, Resistor_SMD:R_0603_1608Metric, F.Cu at (128.0, 86.3)
- added R3: 10k, Resistor_SMD:R_0603_1608Metric, F.Cu at (130.4, 83.9)
- added R4: 300, Resistor_SMD:R_0603_1608Metric, F.Cu at (128.0, 87.9)
- added R5: R, Resistor_SMD:R_2512_6332Metric, F.Cu at (124.4, 88.7)
- added R6: 5.23k, Resistor_SMD:R_0603_1608Metric, F.Cu at (128.0, 84.7)
- added R7: 30.1k, Resistor_SMD:R_0603_1608Metric, F.Cu at (128.0, 83.1)
- added R8: 2.2k, Resistor_SMD:R_0603_1608Metric, F.Cu at (105.0, 88.1)
- added U5: AP63200WU, Package_TO_SOT_SMD:TSOT-23-6, F.Cu at (142.9, 96.3)
- moved U2 244.6 mm to (132.7, 88.1), turned to -90 degrees
- moved U3 235.1 mm to (141.4, 81.9), turned to -90 degrees
- moved U7 176.4 mm to (135.2, 112.9)
- moved U9 164.6 mm to (160.6, 94.7), turned to 90 degrees
- moved C26 135.2 mm to (325.1, 124.1)
- moved L2 53.4 mm to (159.2, 91.3), turned to 180 degrees
- moved C1 49.0 mm to (177.8, 79.2), turned to 180 degrees
- moved C17 48.0 mm to (158.0, 94.8), turned to -90 degrees
- moved C18 47.2 mm to (159.4, 97.6), turned to 180 degrees
- moved DWM1 27.3 mm to (155.3, 72.7)
- moved D3 12.5 mm to (203.5, 133.4), turned to 180 degrees
- moved R15 5.00 mm to (200.4, 133.4)
- moved U1 1.66 mm to (185.9, 81.6)
Connections:
- U2 pad 11: Net-(U2-REGN) -> /Battery Recharger/REGN
- U3 pad 12: Vdrive -> +6V
Routing:
- net /Battery Recharger/TS: track 0.00 -> 8.34 mm
- net Net-(J1-Pin_3): track 0.00 -> 4.65 mm
- net Net-(U5-FB): track 0.00 -> 3.41 mm
- net Net-(U2-ILIM): track 0.00 -> 2.32 mm
- net Net-(U2-MID): track 0.00 -> 1.91 mm
- net /Battery Recharger/~{INT}: track 0.00 -> 1.83 mm
- net Net-(U5-BST): track 0.00 -> 1.80 mm
- net +3V3: track 0.00 -> 0.50 mm
- added copper zone on F.Cu, net +3V3
- added copper zone on F.Cu, net +6V
- added copper zone on F.Cu, net GND
- added copper zone on F.Cu, net Net-(U5-SW)

Commit message: update PCB
Parts:
- added M1: Motor_DC, Connector_JST:JST_PH_B2B-PH-SM4-TB_1x02-1MP_P2.00mm_Vertical, F.Cu at (140.7, 73.6)
- added M2: Motor_DC, Connector_JST:JST_PH_B2B-PH-SM4-TB_1x02-1MP_P2.00mm_Vertical, F.Cu at (131.2, 73.6)
- J1: footprint Connector_JST:JST_PH_S4B-PH-K_1x04_P2.00mm_Horizontal -> Connector_JST:JST_PH_S4B-PH-SM4-TB_1x04-1MP_P2.00mm_Horizontal; moved to B.Cu
- moved D2 30.5 mm to (131.7, 81.5), turned to 90 degrees
- moved D1 29.2 mm to (129.8, 81.5), turned to 90 degrees
- moved R8 27.0 mm to (131.7, 84.6), turned to -90 degrees
- moved R1 25.4 mm to (129.8, 84.6), turned to -90 degrees
- moved U3 5.43 mm to (135.9, 82.0)
- moved J1 5.11 mm to (129.2, 74.5), turned to 0 degrees
- moved C12 3.12 mm to (131.0, 97.5)
- moved C2 3.12 mm to (134.0, 87.7)
- moved C3 3.12 mm to (131.0, 95.1)
- moved C7 3.12 mm to (126.9, 92.8)
- moved R3 3.12 mm to (127.5, 84.9)
- moved C6 3.12 mm to (124.3, 92.3)
- moved R5 3.12 mm to (121.4, 89.7)
- moved R2 3.12 mm to (125.1, 87.3)
- moved R4 3.12 mm to (125.1, 88.9)
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Routing:
- net /Battery Recharger/REGN: track 0.00 -> 4.19 mm
- net /Battery Recharger/TS: track 8.34 -> 4.53 mm
- added copper zone on F.Cu, net Net-(U2-CBSET)
Other:
- board size 78 x 56.6 mm -> 78 x 63.4 mm

Commit message: updates
Parts:
- moved D2 11.0 mm to (121.1, 78.7), turned to 180 degrees
- moved R8 9.56 mm to (124.2, 78.7), turned to 0 degrees
- moved D1 8.80 mm to (121.1, 80.5), turned to 180 degrees
- moved R1 6.96 mm to (124.2, 80.5), turned to 0 degrees
- moved C19 1.39 mm to (137.3, 111.1)
- moved C20 1.31 mm to (142.4, 117.7)
- moved C21 1.31 mm to (142.4, 119.7)
- moved L3 1.31 mm to (141.8, 113.6)
- moved U7 1.31 mm to (136.3, 113.6)
- moved C22 1.10 mm to (136.9, 116.4)
Routing:
- net Net-(U2-~{PG}): track 0.00 -> 12.9 mm
- net Net-(U2-STAT): track 0.00 -> 12.1 mm
- net /Battery Recharger/TS: track 4.53 -> 12.3 mm, vias 0 -> 1
- net Net-(U7-BST): track 0.00 -> 1.94 mm
- net Net-(D2-K): track 0.00 -> 1.50 mm
- net Net-(D1-K): track 0.00 -> 1.49 mm
- net Net-(J1-Pin_3): vias 0 -> 6
- net GND: vias 0 -> 3
- net +5V: vias 0 -> 1
- added copper zone on F.Cu, net +5V
- added copper zone on B.Cu, net Net-(J1-Pin_3)
- added copper zone on F.Cu, net Net-(J1-Pin_3)
- added copper zone on F.Cu, net Net-(U7-SW)

Commit message: more on layout
Parts:
- R5: value R -> 10
- moved C2 0.84 mm to (134.8, 87.7)
Connections:
- net Net-(J1-Pin_3) renamed /Battery Recharger/CBSET_PIN
- net Net-(U2-CBSET) renamed /Battery Recharger/CBSET_IN
Routing:
- net /Battery Recharger/REGN: track 4.19 -> 22.9 mm, vias 0 -> 3
- net /Battery Recharger/CBSET_PIN: track 4.65 -> 20.3 mm, vias 6 -> 2
- net Net-(C12-Pad1): track 0.00 -> 7.01 mm
- net Net-(U2-BTST): track 0.00 -> 6.15 mm, vias 0 -> 2
- net Net-(C4-Pad1): track 0.00 -> 2.31 mm
- net VBUS: track 0.00 -> 0.99 mm, vias 0 -> 4
- net +BATT: vias 0 -> 3
- added copper zone on B.Cu, net +BATT
- added copper zone on F.Cu, net +BATT
- added copper zone on B.Cu, net GND
- added copper zone on B.Cu, net VBUS
- added copper zone on F.Cu, net VBUS
- removed copper zone on B.Cu, net /Battery Recharger/CBSET_PIN
- removed copper zone on F.Cu, net /Battery Recharger/CBSET_PIN

Commit message: updates
Parts:
- L1: footprint Inductor_SMD:L_1008_2520Metric -> Inductor_SMD:L_Sunlord_MWSA0518S
- moved L1 1.96 mm to (137.9, 91.5)
- moved C24 0.64 mm to (146.2, 95.2)
- moved C25 0.64 mm to (147.0, 98.5)
- moved R11 0.64 mm to (139.1, 97.0)
- moved R12 0.64 mm to (140.6, 97.0)
- moved C13 0.63 mm to (142.5, 93.0)
- moved C23 0.63 mm to (148.3, 95.2)
- moved L4 0.63 mm to (146.5, 90.4)
- moved U5 0.63 mm to (143.4, 96.7)
Routing:
- net VBUS: vias 4 -> 3
- net GND: vias 3 -> 5
- added copper zone on F.Cu, net Net-(C4-Pad1)
- added copper zone on F.Cu, net Net-(C5-Pad1)

Commit message: updates
Parts:
- added H3: MountingHole, MountingHole:MountingHole_2.2mm_M2_ISO14580, F.Cu at (191.9, 73.3)
- added H4: MountingHole, MountingHole:MountingHole_2.2mm_M2_ISO14580, F.Cu at (122.4, 73.3)
- added J3: Conn_01x04, Connector_PinSocket_2.54mm:PinSocket_1x04_P2.54mm_Vertical, F.Cu at (153.4, 59.8)
- H1, H2: footprint MountingHole:MountingHole_3.2mm_M3_Pad -> MountingHole:MountingHole_2.2mm_M2_ISO14580
- moved DWM1 31.0 mm to (183.2, 86.2), turned to -90 degrees
- moved C1 21.8 mm to (165.6, 60.5)
- moved U1 21.8 mm to (173.8, 62.9)
- moved J1 13.2 mm to (135.6, 62.9)
- moved M1 13.0 mm to (146.7, 62.1)
- moved M2 13.0 mm to (137.1, 62.1)
- moved U3 11.7 mm to (141.9, 71.8)
- moved H2 2.00 mm to (122.4, 98.7)
- moved H1 2.00 mm to (191.9, 98.7)
Routing:
- net /Battery Recharger/TS: track 12.3 -> 26.5 mm
- net /Battery Recharger/CBSET_PIN: track 20.3 -> 34.5 mm
- net /Battery Recharger/REGN: track 22.9 -> 19.8 mm, vias 3 -> 2
Other:
- board size 78 x 63.4 mm -> 78 x 75.3 mm

Commit message: some progress
Parts:
- H1, H2, H3, H4: footprint MountingHole:MountingHole_2.2mm_M2_ISO14580 -> MountingHole:MountingHole_2.2mm_M2
- M1, M2: footprint Connector_JST:JST_PH_B2B-PH-SM4-TB_1x02-1MP_P2.00mm_Vertical -> Connector_JST:JST_PH_S2B-PH-SM4-TB_1x02-1MP_P2.00mm_Horizontal
- moved C25 15.2 mm to (148.6, 83.4), turned to 90 degrees
- moved C23 13.5 mm to (145.3, 82.1), turned to 0 degrees
- moved C18 13.3 mm to (152.6, 86.2), turned to 0 degrees
- moved C24 11.1 mm to (145.3, 84.1), turned to 0 degrees
- moved U9 10.8 mm to (151.4, 89.2), turned to -90 degrees
- moved U5 10.3 mm to (146.7, 86.9), turned to 180 degrees
- moved R11 9.82 mm to (147.0, 91.3), turned to 0 degrees
- moved R12 9.70 mm to (147.0, 89.7), turned to 180 degrees
- moved L4 8.95 mm to (140.5, 83.8), turned to 90 degrees
- moved C17 7.08 mm to (154.0, 89.0), turned to 90 degrees
- moved L2 6.50 mm to (152.8, 92.6), turned to 0 degrees
- moved C28 5.80 mm to (156.0, 89.0), turned to 90 degrees
- moved C13 5.12 mm to (143.0, 87.9), turned to 180 degrees
- moved U3 2.08 mm to (141.9, 73.9)
- moved M2 0.58 mm to (137.1, 62.7), turned to 180 degrees
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Connections:
- U3 pad 2: Net-(M1--) -> Net-(M1-+)
- U3 pad 4: Net-(M1-+) -> Net-(M1--)
- U3 pad 5: Net-(M2--) -> Net-(M2-+)
- U3 pad 7: Net-(M2-+) -> Net-(M2--)
