File: battery_circuit.kicad_sch (KiCad schematic)
At the start: 22 parts, among them J1 1S2P 18650 Pack, U5 BQ24074RGT, U7 INA219AxD

Commit message: some updates
Parts:
- removed U7: INA219AxD, Package_SO:SOIC-8_3.9x4.9mm_P1.27mm, symbol Sensor_Energy:INA219AxD
- added C25: 0.1uF, Capacitor_SMD:C_0805_2012Metric, symbol Device:C
- added U1: INA219AxDCN, Package_TO_SOT_SMD:SOT-23-8, symbol Sensor_Energy:INA219AxDCN
- TP1, TP2: footprint TestPoint:TestPoint_Pad_D1.5mm -> TestPoint:TestPoint_Pad_D1.0mm
- renumbered D3 to D4
Connections:
- net +3V3: now also C25.1, U1.4 (VS)
- net GND: now also C25.2, U1.3 (GND)
- net IN+: now also U1.1 (IN+)
- net SCL: now also U1.5 (SCL)
- net SDA: now also U1.6 (SDA)
- net VBATT: now also U1.2 (IN-)
- net at JP1.1 (A): now also U1.8 (A1)
- net at JP3.1 (A): now also U1.7 (A0)

Commit message: more on routing
Parts:
- removed JP1: A1, Jumper:SolderJumper-2_P1.3mm_Open_RoundedPad1.0x1.5mm, symbol Jumper:SolderJumper_2_Open
- removed JP3: A0, Jumper:SolderJumper-2_P1.3mm_Open_RoundedPad1.0x1.5mm, symbol Jumper:SolderJumper_2_Open
- removed JP4: Battery Jumper, Jumper:SolderJumper-2_P1.3mm_Bridged2Bar_RoundedPad1.0x1.5mm, symbol Jumper:SolderJumper_2_Bridged
Connections:
- net IN+ is gone; now on net BATT_OUT: R1.2, U1.1 (IN+)
- net GND: now also U1.7 (A0), U1.8 (A1)
