File: rover-circuit.kicad_sch (KiCad schematic)
At the start: 26 parts, among them J2 USB_C_Receptacle_USB2.0_14P, J4 Display Connector, J5 Raspberry_Pi_2_3, J6 Conn_02x07_Odd_Even, SW1 SW_EN, SW2 SW_IO0, U2 ESP32-S3-WROOM-1, U4 TPD2EUSB30

Commit message: start new design
Parts:
- removed C5: 10uF, Capacitor_SMD:C_0805_2012Metric, symbol Device:C
- removed C6: 100uF, Capacitor_SMD:C_0805_2012Metric, symbol Device:C
- removed J2: USB_C_Receptacle_USB2.0_14P, Connector_USB:USB_C_Receptacle_G-Switch_GT-USB-7010ASV, symbol Connector:USB_C_Receptacle_USB2.0_14P
- removed J4: Display Connector, Connector_JST:JST_EH_B8B-EH-A_1x08_P2.50mm_Vertical, symbol Connector:Conn_01x08_Pin
- removed J5: Raspberry_Pi_2_3, Connector_PinSocket_2.54mm:PinSocket_2x20_P2.54mm_Vertical_SMD, symbol Connector:Raspberry_Pi_2_3
- removed J6: Conn_02x07_Odd_Even, Connector_PinHeader_2.54mm:PinHeader_2x07_P2.54mm_Vertical, symbol Connector_Generic:Conn_02x07_Odd_Even
- removed JP2: Disable ESP, Connector_PinHeader_2.54mm:PinHeader_1x02_P2.54mm_Vertical, symbol Jumper:Jumper_2_Open
- removed R12: 100K, Resistor_SMD:R_0805_2012Metric, symbol Device:R
- removed R13, R14: 5.1K, Resistor_SMD:R_0805_2012Metric, symbol Device:R
- removed R2, R6: 4.7K, Resistor_SMD:R_0402_1005Metric, symbol Device:R
- removed SW1: SW_EN, Button_Switch_SMD:SW_SPST_B3U-1000P, symbol Switch:SW_Push
- removed SW2: SW_IO0, Button_Switch_SMD:SW_SPST_B3U-1000P, symbol Switch:SW_Push
- removed TP3: SDA, TestPoint:TestPoint_Pad_D1.0mm, symbol Connector:TestPoint
- removed TP4: SCL, TestPoint:TestPoint_Pad_D1.0mm, symbol Connector:TestPoint
- removed U2: ESP32-S3-WROOM-1, RF_Module:ESP32-S3-WROOM-1U, symbol RF_Module:ESP32-S3-WROOM-1
- removed U4: TPD2EUSB30, Package_TO_SOT_SMD:Texas_DRT-3, symbol Power_Protection:TPD2EUSB30
Connections:
- no-connect marks 4 -> 0
Other:
- removed sheet Battery Circuit
- removed sheet Front Wheels
- removed sheet Motion Tracking
- removed sheet Power Stage
- removed sheet Rear Wheels
- removed sheet UWB Module
- added sheet MCU (mcu.kicad_sch)
- added sheet Rasbpberry PI (sbc.kicad_sch)
- added sheet USB (usb.kicad_sch)
- note removed: "Display Connector"
- note removed: "Motor Drivers"
