File: power_rails.kicad_sch (KiCad schematic)
At the start: 23 parts, among them SW3 SW_Push, U10 LTC2954CDDB-1-PBF, U7 AP63205WU, U8 TPS5430DDA, U9 TPS62162DSG

Commit message: improve design
Connections:
- net +3V3: now also R15.1
Other:
- title: (none) -> Dropbot
- moved on the sheet: C26, SW3, U10

Commit message: design pcb and place components
Parts:
- C17, C18: footprint (none) -> Capacitor_SMD:C_0805_2012Metric
- C26: footprint (none) -> Capacitor_SMD:C_0402_1005Metric
- D3: footprint (none) -> LED_SMD:LED_0603_1608Metric
- L2: footprint (none) -> Inductor_SMD:L_APV_ANR3012
- R15: footprint (none) -> Resistor_SMD:R_0603_1608Metric
Changed lines of the file:
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@@
 			)
 		)
-		(property "Footprint" ""
+		(property "Footprint" "Capacitor_SMD:C_0805_2012Metric"
 			(at 41.6052 165.1 0)
 			(hide yes)
@@
 			)
 		)
-		(property "Footprint" ""
+		(property "Footprint" "Capacitor_SMD:C_0402_1005Metric"
 			(at 242.2652 109.22 0)
 			(hide yes)
@@
 			)
 		)
-		(property "Footprint" ""
+		(property "Footprint" "Inductor_SMD:L_APV_ANR3012"
 			(at 102.87 153.67 0)
 			(hide yes)
@@
 			)
 		)
-		(property "Footprint" ""
+		(property "Footprint" "Capacitor_SMD:C_0805_2012Metric"
 			(at 117.8052 167.64 0)
 			(hide yes)
@@
 			)
 		)
-		(property "Footprint" ""
+		(property "Footprint" "Resistor_SMD:R_0603_1608Metric"
 			(at 58.42 165.608 90)
 			(hide yes)
@@
 			)
 		)
-		(property "Footprint" ""
+		(property "Footprint" "LED_SMD:LED_0603_1608Metric"
 			(at 67.31 163.83 0)
 			(hide yes)

Commit message: moving on routing
Parts:
- removed C25: 220uF, symbol Device:C_Polarized
- removed D4: B340, Diode_SMD:D_SMC, symbol Diode:B340
- removed L4: 15uH, symbol Device:L_Ferrite
- removed R16: 10k, symbol Device:R
- removed R17: 25.5k, symbol Device:R
- removed U8: TPS5430DDA, Package_SO:TI_SO-PowerPAD-8_ThermalVias, symbol Regulator_Switching:TPS5430DDA
- added C13: 100nF, Capacitor_SMD:C_0603_1608Metric, symbol Device:C
- added C25: 10uF, Capacitor_SMD:C_0805_2012Metric, symbol Device:C
- added C28: 22uF, Capacitor_SMD:C_0805_2012Metric, symbol Device:C
- added L4: 10uH, Inductor_SMD:L_Sunlord_MWSA0503S, symbol Device:L
- added R11: 64.9k, Resistor_SMD:R_0603_1608Metric, symbol Device:R
- added R12: 10k, Resistor_SMD:R_0603_1608Metric, symbol Device:R
- added U5: AP63200WU, Package_TO_SOT_SMD:TSOT-23-6, symbol Regulator_Switching:AP63200WU
- C19: footprint (none) -> Capacitor_SMD:C_0603_1608Metric
- C20, C21, C22: footprint (none) -> Capacitor_SMD:C_0805_2012Metric
- C23: value 10uF -> 22uF; footprint (none) -> Capacitor_SMD:C_0805_2012Metric
- C24: value 100nF -> 22uF; footprint (none) -> Capacitor_SMD:C_0805_2012Metric
- L3: footprint (none) -> Inductor_SMD:L_Sunlord_MWSA0503S
Connections:
- net +3V3: now also C28.1
- net +BATT: now also C25.1, U5.3 (IN); no longer C23.1
- net EN: now also U5.2 (EN)
- net GND: now also C24.2, C25.2, C28.2, R12.2, U5.4 (GND)
- net +6V: now reaches C24.1
- net +6V: now also C23.1, L4.2, R11.1
- new net: R11.2, R12.1, U5.1 (FB)
- new net: C13.1, U5.6 (BST)
- new net: C13.2, L4.1, U5.5 (SW)

Commit message: more on routing and schematic
Parts:
- U10: footprint DFN-8_DDB_LIT -> Package_DFN_QFN:DFN-8-1EP_2x3mm_P0.5mm_EP0.61x2.2mm
Changed lines of the file:
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@@
 			)
 		)
-		(property "Footprint" "DFN-8_DDB_LIT"
+		(property "Footprint" "Package_DFN_QFN:DFN-8-1EP_2x3mm_P0.5mm_EP0.61x2.2mm"
 			(at 234.95 88.9 0)
 			(hide yes)

Commit message: updates
Parts:
- SW3: footprint (none) -> Button_Switch_SMD:SW_SPST_B3U-1000P
Other:
- moved on the sheet: C13, C18, C19, C20, C21, C22, C23, C24, C25, L3, L4, R11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

Commit message: complete routing and validated ERC/DRC
Changed lines of the file:
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@@
+	)
+	(symbol
+		(lib_id "power:PWR_FLAG")
+		(at 110.49 153.67 0)
+		(unit 1)
+		(body_style 1)
+		(exclude_from_sim no)
+		(in_bom yes)
+		(on_board yes)
+		(in_pos_files yes)
+		(dnp no)
+		(fields_autoplaced yes)
+		(property "Reference" "#FLG01"
+			(at 110.49 151.765 0)
+			(hide yes)
+			(show_name no)
+			(do_not_autoplace no)
+			(effects
+				(font
+					(size 1.27 1.27)
+				)
+			)
+		)
+		(property "Value" "PWR_FLAG"
+			(at 110.49 148.59 0)
+			(show_name no)
+			(do_not_autoplace no)
+			(effects
+				(font
+					(size 1.27 1.27)
+				)
+			)
+		)
+		(property "Footprint" ""
+			(at 110.49 153.67 0)
+			(hide yes)
+			(show_name no)
+			(do_not_autoplace no)
+			(effects
+				(font
+					(size 1.27 1.27)
+				)
+			)
+		)
+		(property "Datasheet" ""
+			(at 110.49 153.67 0)
+			(hide yes)
+			(show_name no)
+			(do_not_autoplace no)
+			(effects
+				(font
+					(size 1.27 1.27)
+				)
+			)
+		)
+		(property "Description" "Special symbol for telling ERC where power comes from"
+			(at 110.49 153.67 0)
+			(hide yes)
+			(show_name no)
+			(do_not_autoplace no)
+			(effects
+				(font
+					(size 1.27 1.27)
+				)
+			)
+		)
+		(pin "1"
+		)
+		(instances
+			(project "rover-circuit"
+				(path "/0461baee-3b25-4e1a-a5c1-d76b4b99c66c/f4b194fd-8f48-4986-9deb-ce512b0299fe"
+					(reference "#FLG01")
+					(unit 1)
+				)
+			)
+		)
 	)
 	(symbol
@@
 				(path "/0461baee-3b25-4e1a-a5c1-d76b4b99c66c/f4b194fd-8f48-4986-9deb-ce512b0299fe"
 					(reference "C24")
+					(unit 1)
+				)
+			)
+		)
+	)
+	(symbol
+		(lib_id "power:PWR_FLAG")
+		(at 110.49 35.56 0)
+		(unit 1)
+		(body_style 1)
+		(exclude_from_sim no)
+		(in_bom yes)
+		(on_board yes)
+		(in_pos_files yes)
+		(dnp no)
+		(fields_autoplaced yes)
+		(property "Reference" "#FLG03"
+			(at 110.49 33.655 0)
+			(hide yes)
+			(show_name no)
+			(do_not_autoplace no)
+			(effects
+				(font
+					(size 1.27 1.27)
+				)
+			)
+		)
+		(property "Value" "PWR_FLAG"
+			(at 110.49 30.48 0)
+			(show_name no)
+			(do_not_autoplace no)
+			(effects
+				(font
+					(size 1.27 1.27)
+				)
+			)
+		)
+		(property "Footprint" ""
+			(at 110.49 35.56 0)
+			(hide yes)
+			(show_name no)
+			(do_not_autoplace no)
+			(effects
+				(font
+					(size 1.27 1.27)
+				)
+			)
+		)
+		(property "Datasheet" ""
+			(at 110.49 35.56 0)
+			(hide yes)
+			(show_name no)
+			(do_not_autoplace no)
+			(effects
+				(font
+					(size 1.27 1.27)
+				)
+			)
+		)
+		(property "Description" "Special symbol for telling ERC where power comes from"
+			(at 110.49 35.56 0)
+			(hide yes)
+			(show_name no)
+			(do_not_autoplace no)
+			(effects
+				(font
+					(size 1.27 1.27)
+				)
+			)
+		)
+		(pin "1"
+		)
+		(instances
+			(project "rover-circuit"
+				(path "/0461baee-3b25-4e1a-a5c1-d76b4b99c66c/f4b194fd-8f48-4986-9deb-ce512b0299fe"
+					(reference "#FLG03")
 					(unit 1)
 				)
@@
 					(unit 1)
 				)
+			)
+		)
+	)
+	(symbol
+		(lib_id "power:PWR_FLAG")
+		(at 110.49 97.79 0)
+		(unit 1)
+		(body_style 1)
+		(exclude_from_sim no)
+		(in_bom yes)
+		(on_board yes)
+		(in_pos_files yes)
+		(dnp no)
+		(fields_autoplaced yes)
+		(property "Reference" "#FLG02"
+			(at 110.49 95.885 0)
+			(hide yes)
+			(show_name no)
+			(do_not_autoplace no)
+			(effects
+				(font
+					(size 1.27 1.27)
+				)
+			)
+		)
+		(property "Value" "PWR_FLAG"
+			(at 110.49 92.71 0)
+			(show_name no)
+			(do_not_autoplace no)
+			(effects
+				(font
+					(size 1.27 1.27)
+				)
+			)
+		)
+		(property "Footprint" ""
+			(at 110.49 97.79 0)
+			(hide yes)
+			(show_name no)
+			(do_not_autoplace no)
+			(effects
+				(font
+					(size 1.27 1.27)
+				)
+			)
+		)
+		(property "Datasheet" ""
+			(at 110.49 97.79 0)
+			(hide yes)
+			(show_name no)
+			(do_not_autoplace no)
+			(effects
+				(font
+					(size 1.27 1.27)
+				)
+			)
+		)
+		(property "Description" "Special symbol for telling ERC where power comes from"
+			(at 110.49 97.79 0)
+			(hide yes)
+			(show_name no)
+			(do_not_autoplace no)
+			(effects
+				(font
+					(size 1.27 1.27)
+				)
+			)
+		)
+		(pin "1"
+		)
+		(instances
+			(project "rover-circuit"
+				(path "/0461baee-3b25-4e1a-a5c1-d76b4b99c66c/f4b194fd-8f48-4986-9deb-ce512b0299fe"
+					(reference "#FLG02")
+					(unit 1)
+				)

Commit message: tentative automatic population
Parts:
- C13, C19: LCSC (none) -> C14663; MPN (none) -> CC0603KRX7R9BB104; Manufacturer (none) -> YAGEO
- C17, C20, C21, C23, C24, C28: LCSC (none) -> C296720; MPN (none) -> CL21A226KOQNNNE; Manufacturer (none) -> Samsung Electro-Mechanics
- C18, C22, C25: LCSC (none) -> C84416; MPN (none) -> GRM21BR61E106KA73L; Manufacturer (none) -> muRata
- C26: LCSC (none) -> C29266; MPN (none) -> CL05A105KO5NNNC; Manufacturer (none) -> Samsung Electro-Mechanics
- D3: LCSC (none) -> C2286; MPN (none) -> KT-0603R; Manufacturer (none) -> Hubei KENTO Elec
- L2: LCSC (none) -> C2844756; MPN (none) -> LPS3015-222MRC; Manufacturer (none) -> Coilcraft
- L3: LCSC (none) -> C108284; MPN (none) -> LVS505040-4R7M-N; Manufacturer (none) -> Chilisin
- L4: LCSC (none) -> C431344; MPN (none) -> CMLW5040S100MST; Manufacturer (none) -> Cybermax
- R11: LCSC (none) -> C14891; MPN (none) -> 0603WAF6492T5E; Manufacturer (none) -> UNI-ROYAL
- R12: LCSC (none) -> C2906982; MPN (none) -> FRC0603F1002TS; Manufacturer (none) -> FOJAN
- R15: LCSC (none) -> C25803; MPN (none) -> 0603WAF1003T5E; Manufacturer (none) -> UNI-ROYAL
- SW3: LCSC (none) -> C231329; MPN (none) -> B3U-1000P; Manufacturer (none) -> OMRON
- U5: LCSC (none) -> C2071868; MPN (none) -> AP63200WU-7; Manufacturer (none) -> DIODES
- U7: LCSC (none) -> C2071056; MPN (none) -> AP63205WU-7; Manufacturer (none) -> DIODES
- U9: LCSC (none) -> C40256; MPN (none) -> TPS62162DSGR; Manufacturer (none) -> TI

Commit message: Consistent final layout
Parts:
- removed C26: 1uF, Capacitor_SMD:C_0402_1005Metric, symbol Device:C
- removed U10: LTC2954CDDB-1-PBF, Package_DFN_QFN:DFN-8-1EP_2x3mm_P0.5mm_EP0.61x2.2mm, symbol LTC2954CDDB:LTC2954CDDB-1-PBF
- added C32: 1uF, Capacitor_SMD:C_0603_1608Metric, symbol Device:C
- added SW4: ~{PB}, Button_Switch_SMD:SW_SPST_B3U-1000P, symbol Switch:SW_Push
- added U12: MCP1799x-500xxTT, Package_TO_SOT_SMD:SOT-23, symbol Regulator_Linear:MCP1799x-500xxTT
- added U8: STM6601, Package_DFN_QFN:TDFN-12_2x3mm_P0.5mm, symbol Power_Management:STM6601
- SW3: value SW_Push -> ~{SR}
Connections:
- net +BATT: now also U12.3 (VI)
- net EN: now also U8.9 (~{EN}/EN)
- net GND: now also C32.2, SW4.1, U12.1 (GND), U8.12 (GND)
- net at SW3.2: now also U8.2 (~{SR})
- new net: U12.2 (VO), U8.1 (Vcc)
- new net: SW4.2, U8.6 (~{PB})
- new net: C32.1, U8.3 (Vref)
- new net HOLD: U8.4 (PS_HOLD)
- new net PB_OUT: U8.8 (~{PB}_OUT)
- no-connect marks 1 -> 4
Other:
- moved on the sheet: SW3
