File: uwb.kicad_sch (KiCad schematic)
At the start: 7 parts

Commit message: finalized component selection
Parts:
- DWM1: LCSC C95238 -> (none)
- R18: LCSC C2906982 -> C15401; MPN FRC0603F1002TS -> (none); Manufacturer FOJAN -> (none)
Changed lines of the file:
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@@
 			)
 		)
-		(property "Manufacturer" "FOJAN"
-			(at 0 0 0)
-			(hide yes)
-			(show_name no)
-			(do_not_autoplace no)
-			(effects
-				(font
-					(size 1.27 1.27)
-				)
-			)
-		)
-		(property "MPN" "FRC0603F1002TS"
-			(at 0 0 0)
-			(hide yes)
-			(show_name no)
-			(do_not_autoplace no)
-			(effects
-				(font
-					(size 1.27 1.27)
-				)
-			)
-		)
-		(property "LCSC" "C2906982"
+		(property "Manufacturer" ""
+			(at 0 0 0)
+			(hide yes)
+			(show_name no)
+			(do_not_autoplace no)
+			(effects
+				(font
+					(size 1.27 1.27)
+				)
+			)
+		)
+		(property "MPN" ""
+			(at 0 0 0)
+			(hide yes)
+			(show_name no)
+			(do_not_autoplace no)
+			(effects
+				(font
+					(size 1.27 1.27)
+				)
+			)
+		)
+		(property "LCSC" "C15401"
 			(at 0 0 0)
 			(hide yes)
@@
 			)
 		)
-		(property "LCSC" "C95238"
-			(at 0 0 0)
-			(hide yes)
+		(property "LCSC" ""
+			(at 0 0 0)
+			(hide yes)

Commit message: add MPS entries
Parts:
- C27: MPN CC0805KRX7R9BB104 -> GPN; Manufacturer YAGEO -> Generic
- D5, D6: MPN XL-1608UBC-04 -> 150060BS75000; Manufacturer XINGLIGHT -> Wurth Elektronik
- R18: MPN (none) -> GPN; Manufacturer (none) -> Generic
- R19, R20: MPN 0603WAF4700T5E -> GPN; Manufacturer UNI-ROYAL -> Generic
Changed lines of the file:
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@@
 			)
 		)
-		(property "Manufacturer" "XINGLIGHT"
-			(at 0 0 0)
-			(hide yes)
-			(show_name no)
-			(do_not_autoplace no)
-			(effects
-				(font
-					(size 1.27 1.27)
-				)
-			)
-		)
-		(property "MPN" "XL-1608UBC-04"
+		(property "Manufacturer" "Wurth Elektronik"
+			(at 0 0 0)
+			(hide yes)
+			(show_name no)
+			(do_not_autoplace no)
+			(effects
+				(font
+					(size 1.27 1.27)
+				)
+			)
+		)
+		(property "MPN" "150060BS75000"
 			(at 0 0 0)
 			(hide yes)
@@
 			)
 		)
-		(property "Manufacturer" ""
-			(at 0 0 0)
-			(hide yes)
-			(show_name no)
-			(do_not_autoplace no)
-			(effects
-				(font
-					(size 1.27 1.27)
-				)
-			)
-		)
-		(property "MPN" ""
+		(property "Manufacturer" "Generic"
+			(at 0 0 0)
+			(hide yes)
+			(show_name no)
+			(do_not_autoplace no)
+			(effects
+				(font
+					(size 1.27 1.27)
+				)
+			)
+		)
+		(property "MPN" "GPN"
 			(at 0 0 0)
 			(hide yes)
@@
 			)
 		)
-		(property "Manufacturer" "YAGEO"
-			(at 0 0 0)
-			(hide yes)
-			(show_name no)
-			(do_not_autoplace no)
-			(effects
-				(font
-					(size 1.27 1.27)
-				)
-			)
-		)
-		(property "MPN" "CC0805KRX7R9BB104"
+		(property "Manufacturer" "Generic"
+			(at 0 0 0)
+			(hide yes)
+			(show_name no)
+			(do_not_autoplace no)
+			(effects
+				(font
+					(size 1.27 1.27)
+				)
+			)
+		)
+		(property "MPN" "GPN"
 			(at 0 0 0)
 			(hide yes)
@@
 			)
 		)
-		(property "Manufacturer" "XINGLIGHT"
-			(at 0 0 0)
-			(hide yes)
-			(show_name no)
-			(do_not_autoplace no)
-			(effects
-				(font
-					(size 1.27 1.27)
-				)
-			)
-		)
-		(property "MPN" "XL-1608UBC-04"
+		(property "Manufacturer" "Wurth Elektronik"
+			(at 0 0 0)
+			(hide yes)
+			(show_name no)
+			(do_not_autoplace no)
+			(effects
+				(font
+					(size 1.27 1.27)
+				)
+			)
+		)
+		(property "MPN" "150060BS75000"
 			(at 0 0 0)
 			(hide yes)
@@
 			)
 		)
-		(property "Manufacturer" "UNI-ROYAL"
-			(at 0 0 0)
-			(hide yes)
-			(show_name no)
-			(do_not_autoplace no)
-			(effects
-				(font
-					(size 1.27 1.27)
-				)
-			)
-		)
-		(property "MPN" "0603WAF4700T5E"
+		(property "Manufacturer" "Generic"
+			(at 0 0 0)
+			(hide yes)
+			(show_name no)
+			(do_not_autoplace no)
+			(effects
+				(font
+					(size 1.27 1.27)
+				)
+			)
+		)
+		(property "MPN" "GPN"
 			(at 0 0 0)
 			(hide yes)
@@
 			)
 		)
-		(property "Manufacturer" "UNI-ROYAL"
-			(at 0 0 0)
-			(hide yes)
-			(show_name no)
-			(do_not_autoplace no)
-			(effects
-				(font
-					(size 1.27 1.27)
-				)
-			)
-		)
-		(property "MPN" "0603WAF4700T5E"
-			(at 0 0 0)
-			(hide yes)
+		(property "Manufacturer" "Generic"
+			(at 0 0 0)
+			(hide yes)
+			(show_name no)
+			(do_not_autoplace no)
+			(effects
+				(font
+					(size 1.27 1.27)
+				)
+			)
+		)
+		(property "MPN" "GPN"
+			(at 0 0 0)
+			(hide yes)

Commit message: update MPN codes
Parts:
- C27: MPN GPN -> GPC0805104
- R18: MPN GPN -> GPR060310K
- R19, R20: MPN GPN -> GPR0603470R
Changed lines of the file:
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@@
 			)
 		)
-		(property "MPN" "GPN"
+		(property "MPN" "GPR060310K"
 			(at 0 0 0)
 			(hide yes)
@@
 			)
 		)
-		(property "MPN" "GPN"
+		(property "MPN" "GPC0805104"
 			(at 0 0 0)
 			(hide yes)
@@
 			)
 		)
-		(property "MPN" "GPN"
+		(property "MPN" "GPR0603470R"
 			(at 0 0 0)
 			(hide yes)
@@
 			)
 		)
-		(property "MPN" "GPN"
-			(at 0 0 0)
-			(hide yes)
+		(property "MPN" "GPR0603470R"
+			(at 0 0 0)
+			(hide yes)
