File: display.kicad_sch (KiCad schematic)
At the start: 1 part, among them J3 Conn_01x04

Commit message: improve design
Other:
- title: (none) -> Dropbot
Changed lines of the file:
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@@
 	(generator_version "10.0")
 	(paper "A4")
+	(title_block
+		(title "Dropbot")
+	)
 	(bus_entry
 		(at 135.89 92.71)

Commit message: updates
Parts:
- J3: footprint (none) -> Connector_PinSocket_2.54mm:PinSocket_1x04_P2.54mm_Vertical
Changed lines of the file:
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@@
 			)
 		)
-		(property "Footprint" ""
+		(property "Footprint" "Connector_PinSocket_2.54mm:PinSocket_1x04_P2.54mm_Vertical"
 			(at 147.32 95.25 0)
 			(hide yes)

Commit message: some progress
Parts:
- J3: footprint Connector_PinSocket_2.54mm:PinSocket_1x04_P2.54mm_Vertical -> (none)
Changed lines of the file:
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@@
 			)
 		)
-		(property "Footprint" "Connector_PinSocket_2.54mm:PinSocket_1x04_P2.54mm_Vertical"
+		(property "Footprint" ""
 			(at 147.32 95.25 0)
 			(hide yes)

Commit message: annotate with LCSC components
Parts:
- J3: footprint (none) -> Connector_PinSocket_2.54mm:PinSocket_1x04_P2.54mm_Vertical; LCSC (none) -> C2718488; MPN (none) -> 2.54-1*4P; Manufacturer (none) -> BOOMELE(Boom Precision Elec)
Changed lines of the file:
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@@
 			)
 		)
-		(property "Footprint" ""
+		(property "Footprint" "Connector_PinSocket_2.54mm:PinSocket_1x04_P2.54mm_Vertical"
 			(at 147.32 95.25 0)
 			(hide yes)
@@
 			)
 		)
-		(property "Datasheet" ""
+		(property "Datasheet" "https://www.lcsc.com/product-detail/Female-Headers_BOOMELE-Boom-Precision-Elec-2-54-1-4P_C2718488.html"
 			(at 147.32 95.25 0)
 			(hide yes)
@@
 			)
 		)
+		(property "LCSC" "C2718488" (at 0 0 0)
+			(effects
+				(font
+					(size 1.27 1.27)
+				)
+				(hide yes)
+			)
+		)
+		(property "MPN" "2.54-1*4P" (at 0 0 0)
+			(effects
+				(font
+					(size 1.27 1.27)
+				)
+				(hide yes)
+			)
+		)
+		(property "Manufacturer" "BOOMELE(Boom Precision Elec)" (at 0 0 0)
+			(effects
+				(font
+					(size 1.27 1.27)
+				)
+				(hide yes)
+			)
+		)

Commit message: finalized component selection
Parts:
- J3: value Conn_01x04 -> OLED Display
Changed lines of the file:
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@@
 			)
 		)
-		(property "Value" "Conn_01x04"
+		(property "Value" "OLED Display"
 			(at 149.86 97.7899 0)
 			(show_name no)

Commit message: add MPS entries
Parts:
- J3: MPN 2.54-1*4P -> PPTC041LFBN-RC; Manufacturer BOOMELE(Boom Precision Elec) -> Sullins Connector Solutions
Changed lines of the file:
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@@
 			)
 		)
-		(property "MPN" "2.54-1*4P"
+		(property "MPN" "PPTC041LFBN-RC"
 			(at 0 0 0)
 			(hide yes)
@@
 			)
 		)
-		(property "Manufacturer" "BOOMELE(Boom Precision Elec)"
+		(property "Manufacturer" "Sullins Connector Solutions"
 			(at 0 0 0)
 			(hide yes)
