File: recharger.kicad_sch (KiCad schematic)
At the start: 20 parts, among them J1 Battery Connector, U2 BQ25887RGE

Commit message: tentative automatic population
Parts:
- added C16: 1uF, Capacitor_SMD:C_0603_1608Metric, symbol Device:C
- C12, C3: LCSC (none) -> C77091; MPN (none) -> GRM31CR61E226KE15L; Manufacturer (none) -> muRata
- C2: LCSC (none) -> C5673; MPN (none) -> CL10A105KA8NNNC; Manufacturer (none) -> Samsung Electro-Mechanics
- C4: LCSC (none) -> C1622; MPN (none) -> CL10B473KB8NNNC; Manufacturer (none) -> Samsung Electro-Mechanics
- C5: LCSC (none) -> C13585; MPN (none) -> CL31A106KBHNNNE; Manufacturer (none) -> Samsung Electro-Mechanics
- C6: LCSC (none) -> C69335; MPN (none) -> CL10A475KA8NQNC; Manufacturer (none) -> Samsung Electro-Mechanics
- C7: LCSC (none) -> C84416; MPN (none) -> GRM21BR61E106KA73L; Manufacturer (none) -> muRata
- D1: LCSC (none) -> C2286; MPN (none) -> KT-0603R; Manufacturer (none) -> Hubei KENTO Elec
- D2: LCSC (none) -> C965805; MPN (none) -> XL-1608SYGC-06; Manufacturer (none) -> XINGLIGHT
- J1: LCSC (none) -> C265102; MPN (none) -> S4B-PH-SM4-TB(LF)(SN); Manufacturer (none) -> JST
- L1: LCSC (none) -> C167216; MPN (none) -> FXL0630-1R0-M; Manufacturer (none) -> cjiang
- R1, R8: LCSC (none) -> C4190; MPN (none) -> 0603WAF2201T5E; Manufacturer (none) -> UNI-ROYAL
- R2: LCSC (none) -> C22764; MPN (none) -> 0603WAF1101T5E; Manufacturer (none) -> UNI-ROYAL
- R3: LCSC (none) -> C2906982; MPN (none) -> FRC0603F1002TS; Manufacturer (none) -> FOJAN
- R4: LCSC (none) -> C2930092; MPN (none) -> FRC0603F3000TS; Manufacturer (none) -> FOJAN
- R5: LCSC (none) -> C2934046; MPN (none) -> FRC2512F10R0TS; Manufacturer (none) -> FOJAN
- R6: LCSC (none) -> C23068; MPN (none) -> 0603WAF5231T5E; Manufacturer (none) -> UNI-ROYAL
- R7: LCSC (none) -> C23000; MPN (none) -> 0603WAF3012T5E; Manufacturer (none) -> UNI-ROYAL
- U2: LCSC (none) -> C2761614; MPN (none) -> BQ25887RGER; Manufacturer (none) -> TI
Connections:
- net GND: now also C16.2
- net VBUS: now also C16.1

Commit message: Consistent final layout
Parts:
- removed J1: Battery Connector, Connector_JST:JST_PH_S4B-PH-SM4-TB_1x04-1MP_P2.00mm_Horizontal, symbol Connector:Conn_01x04_Pin
- added J9: Battery Connector, Connector_JST:JST_PH_S4B-PH-SM4-TB_1x04-1MP_P2.00mm_Horizontal, symbol Connector_Generic_MountingPin:Conn_01x04_MountingPin
Connections:
- net +BATT: now also J9.4 (Pin_4)
- net CBSET_PIN: now also J9.3 (Pin_3)
- net GND: now also J9.1 (Pin_1)
- net TS: now also J9.2 (Pin_2)
- no-connect marks 2 -> 3

Commit message: annotate with LCSC components
Parts:
- J9: LCSC (none) -> C265102; MPN (none) -> S4B-PH-SM4-TB(LF)(SN); Manufacturer (none) -> JST
Changed lines of the file:
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@@
 			)
 		)
-		(property "Datasheet" ""
+		(property "Datasheet" "https://datasheet.lcsc.com/datasheet/pdf/6c6fce4367275d84ec6a99bf09f1250f.pdf?productCode=C265102"
 			(at 194.31 109.22 0)
 			(hide yes)
@@
 			)
 		)
+		(property "LCSC" "C265102" (at 0 0 0)
+			(effects
+				(font
+					(size 1.27 1.27)
+				)
+				(hide yes)
+			)
+		)
+		(property "MPN" "S4B-PH-SM4-TB(LF)(SN)" (at 0 0 0)
+			(effects
+				(font
+					(size 1.27 1.27)
+				)
+				(hide yes)
+			)
+		)
+		(property "Manufacturer" "JST" (at 0 0 0)
+			(effects
+				(font
+					(size 1.27 1.27)
+				)
+				(hide yes)
+			)
+		)

Commit message: changed power layout
Parts:
- J9: footprint Connector_JST:JST_PH_S4B-PH-SM4-TB_1x04-1MP_P2.00mm_Horizontal -> Connector_JST:JST_SH_BM04B-SRSS-TB_1x04-1MP_P1.00mm_Vertical; LCSC C265102 -> (none)
Changed lines of the file:
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@@
 			)
 		)
-		(property "Footprint" "Connector_JST:JST_PH_S4B-PH-SM4-TB_1x04-1MP_P2.00mm_Horizontal"
+		(property "Footprint" "Connector_JST:JST_SH_BM04B-SRSS-TB_1x04-1MP_P1.00mm_Vertical"
 			(at 194.31 109.22 0)
 			(hide yes)
@@
 			)
 		)
-		(property "LCSC" "C265102" (at 0 0 0)
+		(property "LCSC" ""
+			(at 0 0 0)
+			(hide yes)
+			(show_name no)
+			(do_not_autoplace no)
 			(effects
 				(font
 					(size 1.27 1.27)
 				)
-				(hide yes)
 			)
 		)
-		(property "MPN" "S4B-PH-SM4-TB(LF)(SN)" (at 0 0 0)
+		(property "MPN" "S4B-PH-SM4-TB(LF)(SN)"
+			(at 0 0 0)
+			(hide yes)
+			(show_name no)
+			(do_not_autoplace no)
 			(effects
 				(font
 					(size 1.27 1.27)
 				)
-				(hide yes)
 			)
 		)
-		(property "Manufacturer" "JST" (at 0 0 0)
+		(property "Manufacturer" "JST"
+			(at 0 0 0)
+			(hide yes)
+			(show_name no)
+			(do_not_autoplace no)
 			(effects
 				(font
 					(size 1.27 1.27)
 				)
-				(hide yes)
 			)
 		)

Commit message: optimized space
Parts:
- C7: footprint Capacitor_SMD:C_0805_2012Metric -> Capacitor_SMD:C_0603_1608Metric; LCSC C84416 -> (none); MPN GRM21BR61E106KA73L -> (none); Manufacturer muRata -> (none)
- J9: footprint Connector_JST:JST_SH_BM04B-SRSS-TB_1x04-1MP_P1.00mm_Vertical -> Connector_JST:JST_PH_B4B-PH-SM4-TB_1x04-1MP_P2.00mm_Vertical
Changed lines of the file:
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@@
 			)
 		)
-		(property "Footprint" "Connector_JST:JST_SH_BM04B-SRSS-TB_1x04-1MP_P1.00mm_Vertical"
+		(property "Footprint" "Connector_JST:JST_PH_B4B-PH-SM4-TB_1x04-1MP_P2.00mm_Vertical"
 			(at 194.31 109.22 0)
 			(hide yes)
@@
 			)
 		)
-		(property "Footprint" "Capacitor_SMD:C_0805_2012Metric"
+		(property "Footprint" "Capacitor_SMD:C_0603_1608Metric"
 			(at 207.9752 90.17 0)
 			(hide yes)
@@
 			)
 		)
-		(property "Manufacturer" "muRata"
-			(at 0 0 0)
-			(hide yes)
-			(show_name no)
-			(do_not_autoplace no)
-			(effects
-				(font
-					(size 1.27 1.27)
-				)
-			)
-		)
-		(property "MPN" "GRM21BR61E106KA73L"
-			(at 0 0 0)
-			(hide yes)
-			(show_name no)
-			(do_not_autoplace no)
-			(effects
-				(font
-					(size 1.27 1.27)
-				)
-			)
-		)
-		(property "LCSC" "C84416"
-			(at 0 0 0)
-			(hide yes)
+		(property "Manufacturer" ""
+			(at 0 0 0)
+			(hide yes)
+			(show_name no)
+			(do_not_autoplace no)
+			(effects
+				(font
+					(size 1.27 1.27)
+				)
+			)
+		)
+		(property "MPN" ""
+			(at 0 0 0)
+			(hide yes)
+			(show_name no)
+			(do_not_autoplace no)
+			(effects
+				(font
+					(size 1.27 1.27)
+				)
+			)
+		)
+		(property "LCSC" ""
+			(at 0 0 0)
+			(hide yes)

Commit message: finalized board
Parts:
- added TP6: Batt, TestPoint:TestPoint_Pad_D1.0mm, symbol Connector:TestPoint
- C7: LCSC (none) -> C962136; MPN (none) -> CL10A106KO8NQNC; Manufacturer (none) -> Samsung Electro-Mechanics
- J9: LCSC (none) -> C160354; MPN S4B-PH-SM4-TB(LF)(SN) -> B4B-PH-SM4-TB(LF)(SN)
- R5: LCSC C2934046 -> C1870255; MPN FRC2512F10R0TS -> (none); Manufacturer FOJAN -> (none)
Connections:
- net +BATT: now also TP6.1
Changed lines of the file:
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@@
 	)
 	(junction
+		(at 181.61 104.14)
+		(diameter 0)
+		(color 0 0 0 0)
+	)
+	(junction
 		(at 158.75 121.92)
 		(diameter 0)
@@
 	(wire
 		(pts
+			(xy 181.61 104.14) (xy 186.69 104.14)
+		)
+		(stroke
+			(width 0)
+			(type default)
+		)
+	)
+	(wire
+		(pts
 			(xy 152.4 81.28) (xy 167.64 81.28)
 		)
@@
 	(wire
 		(pts
+			(xy 181.61 96.52) (xy 181.61 104.14)
+		)
+		(stroke
+			(width 0)
+			(type default)
+		)
+	)
+	(wire
+		(pts
 			(xy 152.4 116.84) (xy 154.94 116.84)
 		)
@@
 	(wire
 		(pts
-			(xy 176.53 104.14) (xy 186.69 104.14)
+			(xy 176.53 104.14) (xy 181.61 104.14)
 		)
 		(stroke
@@
 			)
 		)
-		(property "Datasheet" "https://datasheet.lcsc.com/datasheet/pdf/6c6fce4367275d84ec6a99bf09f1250f.pdf?productCode=C265102"
+		(property "Datasheet" "https://lcsc.com/datasheet/lcsc_datasheet_2304140030_JST-B4B-PH-SM4-TB-LF-SN_C160354.pdf"
 			(at 194.31 109.22 0)
 			(hide yes)
@@
 			)
 		)
-		(property "LCSC" ""
+		(property "LCSC" "C160354"
 			(at 0 0 0)
 			(hide yes)
@@
 			)
 		)
-		(property "MPN" "S4B-PH-SM4-TB(LF)(SN)"
+		(property "MPN" "B4B-PH-SM4-TB(LF)(SN)"
 			(at 0 0 0)
 			(hide yes)
@@
 			)
 		)
-		(property "Datasheet" "https://datasheet.lcsc.com/datasheet/pdf/7bcffd7e105d4d878e7542545928cdd2.pdf?productCode=C84416"
+		(property "Datasheet" "https://datasheet.lcsc.com/datasheet/pdf/02336ea48ea44ca18c72517dd3cb7b47.pdf?productCode=C962136"
 			(at 207.01 86.36 0)
 			(hide yes)
@@
 			)
 		)
-		(property "Manufacturer" ""
+		(property "Manufacturer" "Samsung Electro-Mechanics"
 			(at 0 0 0)
 			(hide yes)
@@
 			)
 		)
-		(property "MPN" ""
+		(property "MPN" "CL10A106KO8NQNC"
 			(at 0 0 0)
 			(hide yes)
@@
 			)
 		)
-		(property "LCSC" ""
+		(property "LCSC" "C962136"
 			(at 0 0 0)
 			(hide yes)
@@
 	)
 	(symbol
+		(lib_id "Connector:TestPoint")
+		(at 181.61 96.52 0)
+		(unit 1)
+		(body_style 1)
+		(exclude_from_sim no)
+		(in_bom yes)
+		(on_board yes)
+		(in_pos_files yes)
+		(dnp no)
+		(fields_autoplaced yes)
+		(property "Reference" "TP6"
+			(at 184.15 91.9479 0)
+			(show_name no)
+			(do_not_autoplace no)
+			(effects
+				(font
+					(size 1.27 1.27)
+				)
+				(justify left)
+			)
+		)
+		(property "Value" "Batt"
+			(at 184.15 94.4879 0)
+			(show_name no)
+			(do_not_autoplace no)
+			(effects
+				(font
+					(size 1.27 1.27)
+				)
+				(justify left)
+			)
+		)
+		(property "Footprint" "TestPoint:TestPoint_Pad_D1.0mm"
+			(at 186.69 96.52 0)
+			(hide yes)
+			(show_name no)
+			(do_not_autoplace no)
+			(effects
+				(font
+					(size 1.27 1.27)
+				)
+			)
+		)
+		(property "Datasheet" ""
+			(at 186.69 96.52 0)
+			(hide yes)
+			(show_name no)
+			(do_not_autoplace no)
+			(effects
+				(font
+					(size 1.27 1.27)
+				)
+			)
+		)
+		(property "Description" "test point"
+			(at 181.61 96.52 0)
+			(hide yes)
+			(show_name no)
+			(do_not_autoplace no)
+			(effects
+				(font
+					(size 1.27 1.27)
+				)
+			)
+		)
+		(pin "1"
+		)
+		(instances
+			(project "rover-circuit"
+				(path "/0461baee-3b25-4e1a-a5c1-d76b4b99c66c/d12ae2b7-4c48-4e18-8e74-760d158fba59"
+					(reference "TP6")
+					(unit 1)
+				)
+			)
+		)
+	)
+	(symbol
 		(lib_id "Device:R")
 		(at 158.75 116.84 0)
@@
 			)
 		)
-		(property "Manufacturer" "FOJAN"
+		(property "Manufacturer" ""
 			(at 0 0 0)
 			(hide yes)
@@
 			)
 		)
-		(property "MPN" "FRC2512F10R0TS"
+		(property "MPN" ""
 			(at 0 0 0)
 			(hide yes)
@@
 			)
 		)
-		(property "LCSC" "C2934046"
+		(property "LCSC" "C1870255"
 			(at 0 0 0)
 			(hide yes)

Commit message: finalized component selection
Parts:
- added R21: 10k, Resistor_SMD:R_0603_1608Metric, symbol Device:R
- C7: value 10uF -> 22uF; LCSC C962136 -> C29519229; MPN CL10A106KO8NQNC -> (none); Manufacturer Samsung Electro-Mechanics -> (none)
- L1: LCSC C167216 -> C475532; MPN FXL0630-1R0-M -> (none)
- R3: LCSC C2906982 -> C15401; MPN FRC0603F1002TS -> (none); Manufacturer FOJAN -> (none)
- R5: LCSC C1870255 -> C840605
Connections:
- net REGN: now also R21.1
- net at U2.24 (PSEL): now also R21.2
- no-connect marks 3 -> 2
Changed lines of the file:
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@@
 	)
 	(junction
+		(at 99.06 101.6)
+		(diameter 0)
+		(color 0 0 0 0)
+	)
+	(junction
 		(at 158.75 121.92)
 		(diameter 0)
@@
 		(at 132.08 106.68)
 	)
-	(no_connect
-		(at 132.08 104.14)
-	)
 	(bus_entry
 		(at 106.68 93.98)
@@
 	(wire
 		(pts
-			(xy 93.98 101.6) (xy 100.33 101.6)
+			(xy 93.98 101.6) (xy 99.06 101.6)
 		)
 		(stroke
@@
 	(wire
 		(pts
+			(xy 121.92 104.14) (xy 132.08 104.14)
+		)
+		(stroke
+			(width 0)
+			(type default)
+		)
+	)
+	(wire
+		(pts
 			(xy 176.53 99.06) (xy 176.53 104.14)
 		)
@@
 		)
 	)
+	(wire
+		(pts
+			(xy 99.06 104.14) (xy 99.06 101.6)
+		)
+		(stroke
+			(width 0)
+			(type default)
+		)
+	)
 	(bus
 		(pts
@@
 	(wire
 		(pts
+			(xy 99.06 101.6) (xy 100.33 101.6)
+		)
+		(stroke
+			(width 0)
+			(type default)
+		)
+	)
+	(wire
+		(pts
 			(xy 105.41 114.3) (xy 116.84 114.3)
 		)
@@
 	(wire
 		(pts
+			(xy 114.3 104.14) (xy 99.06 104.14)
+		)
+		(stroke
+			(width 0)
+			(type default)
+		)
+	)
+	(wire
+		(pts
 			(xy 152.4 106.68) (xy 156.21 106.68)
 		)
@@
 			)
 		)
-		(property "Manufacturer" "FOJAN"
+		(property "Manufacturer" ""
 			(at 0 0 0)
 			(hide yes)
@@
 			)
 		)
-		(property "MPN" "FRC0603F1002TS"
+		(property "MPN" ""
 			(at 0 0 0)
 			(hide yes)
@@
 			)
 		)
-		(property "LCSC" "C2906982"
+		(property "LCSC" "C15401"
 			(at 0 0 0)
 			(hide yes)
@@
 			)
 		)
-		(property "MPN" "FXL0630-1R0-M"
+		(property "MPN" ""
 			(at 0 0 0)
 			(hide yes)
@@
 			)
 		)
-		(property "LCSC" "C167216"
+		(property "LCSC" "C475532"
 			(at 0 0 0)
 			(hide yes)
@@
 			)
 		)
-		(property "Value" "10uF"
+		(property "Value" "22uF"
 			(at 210.82 87.6299 0)
 			(show_name no)
@@
 			)
 		)
-		(property "Manufacturer" "Samsung Electro-Mechanics"
+		(property "Manufacturer" ""
 			(at 0 0 0)
 			(hide yes)
@@
 			)
 		)
-		(property "MPN" "CL10A106KO8NQNC"
+		(property "MPN" ""
 			(at 0 0 0)
 			(hide yes)
@@
 			)
 		)
-		(property "LCSC" "C962136"
+		(property "LCSC" "C29519229"
 			(at 0 0 0)
 			(hide yes)
@@
 	)
 	(symbol
+		(lib_id "Device:R")
+		(at 118.11 104.14 90)
+		(unit 1)
+		(body_style 1)
+		(exclude_from_sim no)
+		(in_bom yes)
+		(on_board yes)
+		(in_pos_files yes)
+		(dnp no)
+		(fields_autoplaced yes)
+		(property "Reference" "R21"
+			(at 118.11 97.79 90)
+			(show_name no)
+			(do_not_autoplace no)
+			(effects
+				(font
+					(size 1.27 1.27)
+				)
+			)
+		)
+		(property "Value" "10k"
+			(at 118.11 100.33 90)
+			(show_name no)
+			(do_not_autoplace no)
+			(effects
+				(font
+					(size 1.27 1.27)
+				)
+			)
+		)
+		(property "Footprint" "Resistor_SMD:R_0603_1608Metric"
+			(at 118.11 105.918 90)
+			(hide yes)
+			(show_name no)
+			(do_not_autoplace no)
+			(effects
+				(font
+					(size 1.27 1.27)
+				)
+			)
+		)
+		(property "Datasheet" "https://datasheet.lcsc.com/datasheet/pdf/b3641306390dfb6f98ec07837c926b58.pdf?productCode=C2906982"
+			(at 118.11 104.14 0)
+			(hide yes)
+			(show_name no)
+			(do_not_autoplace no)
+			(effects
+				(font
+					(size 1.27 1.27)
+				)
+			)
+		)
+		(property "Description" "Resistor"
+			(at 118.11 104.14 0)
+			(hide yes)
+			(show_name no)
+			(do_not_autoplace no)
+			(effects
+				(font
+					(size 1.27 1.27)
+				)
+			)
+		)
+		(property "Manufacturer" ""
+			(at 13.97 2.54 0)
+			(hide yes)
+			(show_name no)
+			(do_not_autoplace no)
+			(effects
+				(font
+					(size 1.27 1.27)
+				)
+			)
+		)
+		(property "MPN" ""
+			(at 13.97 2.54 0)
+			(hide yes)
+			(show_name no)
+			(do_not_autoplace no)
+			(effects
+				(font
+					(size 1.27 1.27)
+				)
+			)
+		)
+		(property "LCSC" "C15401"
+			(at 13.97 2.54 0)
+			(hide yes)
+			(show_name no)
+			(do_not_autoplace no)
+			(effects
+				(font
+					(size 1.27 1.27)
+				)
+			)
+		)
+		(pin "1"
+		)
+		(pin "2"
+		)
+		(instances
+			(project "rover-circuit"
+				(path "/0461baee-3b25-4e1a-a5c1-d76b4b99c66c/d12ae2b7-4c48-4e18-8e74-760d158fba59"
+					(reference "R21")
+					(unit 1)
+				)
+			)
+		)
+	)
+	(symbol
 		(lib_id "power:GND")
 		(at 127 127 0)
@@
 			)
 		)
-		(property "LCSC" "C1870255"
+		(property "LCSC" "C840605"
 			(at 0 0 0)
 			(hide yes)

Commit message: add MPS entries
Parts:
- C12, C3: MPN GRM31CR61E226KE15L -> GPN; Manufacturer muRata -> Generic
- C16, C2: MPN CL10A105KA8NNNC -> GPN; Manufacturer Samsung Electro-Mechanics -> Generic
- C4: MPN CL10B473KB8NNNC -> GPN; Manufacturer Samsung Electro-Mechanics -> Generic
- C5: MPN CL31A106KBHNNNE -> GPN; Manufacturer Samsung Electro-Mechanics -> Generic
- C6: MPN CL10A475KA8NQNC -> GPN; Manufacturer Samsung Electro-Mechanics -> Generic
- C7: MPN (none) -> GRM188C61E226ME01D; Manufacturer (none) -> Murata
- D1: MPN KT-0603R -> 150060RS75000; Manufacturer Hubei KENTO Elec -> Wurth Elektronik
- D2: MPN XL-1608SYGC-06 -> 150060VS75000; Manufacturer XINGLIGHT -> Wurth Elektronik
- R1, R8: MPN 0603WAF2201T5E -> GPN; Manufacturer UNI-ROYAL -> Generic
- R2: MPN 0603WAF1101T5E -> GPN; Manufacturer UNI-ROYAL -> Generic
- R21, R3: MPN (none) -> GPN; Manufacturer (none) -> Generic
- R4: MPN FRC0603F3000TS -> GPN; Manufacturer FOJAN -> Generic
- R5: MPN (none) -> CRM2512-FX-10R0ELF; Manufacturer (none) -> Bourns
- R6: MPN 0603WAF5231T5E -> GPN; Manufacturer UNI-ROYAL -> Generic
- R7: MPN 0603WAF3012T5E -> GPN; Manufacturer UNI-ROYAL -> Generic
Changed lines of the file:
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@@
 			)
 		)
-		(property "Manufacturer" ""
+		(property "Manufacturer" "Generic"
 			(at 0 0 0)
 			(hide yes)
@@
 			)
 		)
-		(property "MPN" ""
+		(property "MPN" "GPN"
 			(at 0 0 0)
 			(hide yes)
@@
 			)
 		)
-		(property "Manufacturer" "Samsung Electro-Mechanics"
+		(property "Manufacturer" "Generic"
 			(at 0 0 0)
 			(hide yes)
@@
 			)
 		)
-		(property "MPN" "CL10A105KA8NNNC"
+		(property "MPN" "GPN"
 			(at 0 0 0)
 			(hide yes)
@@
 			)
 		)
-		(property "Manufacturer" "XINGLIGHT"
+		(property "Manufacturer" "Wurth Elektronik"
 			(at 0 0 0)
 			(hide yes)
@@
 			)
 		)
-		(property "MPN" "XL-1608SYGC-06"
+		(property "MPN" "150060VS75000"
 			(at 0 0 0)
 			(hide yes)
@@
 			)
 		)
-		(property "Manufacturer" "UNI-ROYAL"
+		(property "Manufacturer" "Generic"
 			(at 0 0 0)
 			(hide yes)
@@
 			)
 		)
-		(property "MPN" "0603WAF2201T5E"
+		(property "MPN" "GPN"
 			(at 0 0 0)
 			(hide yes)
@@
 			)
 		)
-		(property "Manufacturer" "Hubei KENTO Elec"
+		(property "Manufacturer" "Wurth Elektronik"
 			(at 0 0 0)
 			(hide yes)
@@
 			)
 		)
-		(property "MPN" "KT-0603R"
+		(property "MPN" "150060RS75000"
 			(at 0 0 0)
 			(hide yes)
@@
 			)
 		)
-		(property "Manufacturer" "Samsung Electro-Mechanics"
+		(property "Manufacturer" "Generic"
 			(at 0 0 0)
 			(hide yes)
@@
 			)
 		)
-		(property "MPN" "CL10A105KA8NNNC"
+		(property "MPN" "GPN"
 			(at 0 0 0)
 			(hide yes)
@@
 			)
 		)
-		(property "Manufacturer" "muRata"
+		(property "Manufacturer" "Generic"
 			(at 0 0 0)
 			(hide yes)
@@
 			)
 		)
-		(property "MPN" "GRM31CR61E226KE15L"
+		(property "MPN" "GPN"
 			(at 0 0 0)
 			(hide yes)
@@
 			)
 		)
-		(property "Manufacturer" ""
+		(property "Manufacturer" "Murata"
 			(at 0 0 0)
 			(hide yes)
@@
 			)
 		)
-		(property "MPN" ""
+		(property "MPN" "GRM188C61E226ME01D"
 			(at 0 0 0)
 			(hide yes)
@@
 			)
 		)
-		(property "Manufacturer" "UNI-ROYAL"
+		(property "Manufacturer" "Generic"
 			(at 0 0 0)
 			(hide yes)
@@
 			)
 		)
-		(property "MPN" "0603WAF1101T5E"
+		(property "MPN" "GPN"
 			(at 0 0 0)
 			(hide yes)
@@
 			)
 		)
-		(property "Manufacturer" ""
+		(property "Manufacturer" "Generic"
 			(at 13.97 2.54 0)
 			(hide yes)
@@
 			)
 		)
-		(property "MPN" ""
+		(property "MPN" "GPN"
 			(at 13.97 2.54 0)
 			(hide yes)
@@
 			)
 		)
-		(property "Manufacturer" "Samsung Electro-Mechanics"
+		(property "Manufacturer" "Generic"
 			(at 0 0 0)
 			(hide yes)
@@
 			)
 		)
-		(property "MPN" "CL31A106KBHNNNE"
+		(property "MPN" "GPN"
 			(at 0 0 0)
 			(hide yes)
@@
 			)
 		)
-		(property "Manufacturer" "Samsung Electro-Mechanics"
+		(property "Manufacturer" "Generic"
 			(at 0 0 0)
 			(hide yes)
@@
 			)
 		)
-		(property "MPN" "CL10A475KA8NQNC"
+		(property "MPN" "GPN"
 			(at 0 0 0)
 			(hide yes)
@@
 			)
 		)
-		(property "Manufacturer" "UNI-ROYAL"
+		(property "Manufacturer" "Generic"
 			(at 0 0 0)
 			(hide yes)
@@
 			)
 		)
-		(property "MPN" "0603WAF3012T5E"
+		(property "MPN" "GPN"
 			(at 0 0 0)
 			(hide yes)
@@
 			)
 		)
-		(property "Manufacturer" "muRata"
+		(property "Manufacturer" "Generic"
 			(at 0 0 0)
 			(hide yes)
@@
 			)
 		)
-		(property "MPN" "GRM31CR61E226KE15L"
+		(property "MPN" "GPN"
 			(at 0 0 0)
 			(hide yes)
@@
 			)
 		)
-		(property "Manufacturer" "Samsung Electro-Mechanics"
+		(property "Manufacturer" "Generic"
 			(at 0 0 0)
 			(hide yes)
@@
 			)
 		)
-		(property "MPN" "CL10B473KB8NNNC"
+		(property "MPN" "GPN"
 			(at 0 0 0)
 			(hide yes)
@@
 			)
 		)
-		(property "Manufacturer" "UNI-ROYAL"
+		(property "Manufacturer" "Generic"
 			(at 0 0 0)
 			(hide yes)
@@
 			)
 		)
-		(property "MPN" "0603WAF5231T5E"
+		(property "MPN" "GPN"
 			(at 0 0 0)
 			(hide yes)
@@
 			)
 		)
-		(property "Manufacturer" ""
+		(property "Manufacturer" "Bourns"
 			(at 0 0 0)
 			(hide yes)
@@
 			)
 		)
-		(property "MPN" ""
+		(property "MPN" "CRM2512-FX-10R0ELF"
 			(at 0 0 0)
 			(hide yes)
@@
 			)
 		)
-		(property "Manufacturer" "FOJAN"
+		(property "Manufacturer" "Generic"
 			(at 0 0 0)
 			(hide yes)
@@
 			)
 		)
-		(property "MPN" "FRC0603F3000TS"
+		(property "MPN" "GPN"
 			(at 0 0 0)
 			(hide yes)
@@
 			)
 		)
-		(property "Manufacturer" "UNI-ROYAL"
+		(property "Manufacturer" "Generic"
 			(at 0 0 0)
 			(hide yes)
@@
 			)
 		)
-		(property "MPN" "0603WAF2201T5E"
+		(property "MPN" "GPN"
 			(at 0 0 0)
 			(hide yes)
