File: recharger.kicad_sch (KiCad schematic)
At the start: 23 parts, among them J9 Battery Connector, U2 BQ25887RGE

Commit message: update MPN codes
Parts:
- C12, C3: MPN GPN -> GPC1206226
- C16, C2: MPN GPN -> GPC0603105
- C4: MPN GPN -> GPC0603473
- C5: MPN GPN -> GPC1206106
- C6: MPN GPN -> GPC0603475
- R1, R8: MPN GPN -> GPR060322
- R2: MPN GPN -> GPR060311
- R21, R3: MPN GPN -> GPR060310K
- R4: MPN GPN -> GPR0603300R
- R6: MPN GPN -> GPR0603523
- R7: MPN GPN -> GPR0603301
Changed lines of the file:
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@@
 			)
 		)
-		(property "MPN" "GPN"
+		(property "MPN" "GPR060310K"
 			(at 0 0 0)
 			(hide yes)
@@
 			)
 		)
-		(property "MPN" "GPN"
+		(property "MPN" "GPC0603105"
 			(at 0 0 0)
 			(hide yes)
@@
 			)
 		)
-		(property "MPN" "GPN"
+		(property "MPN" "GPR060322"
 			(at 0 0 0)
 			(hide yes)
@@
 			)
 		)
-		(property "MPN" "GPN"
+		(property "MPN" "GPC0603105"
 			(at 0 0 0)
 			(hide yes)
@@
 			)
 		)
-		(property "MPN" "GPN"
+		(property "MPN" "GPC1206226"
 			(at 0 0 0)
 			(hide yes)
@@
 			)
 		)
-		(property "MPN" "GPN"
+		(property "MPN" "GPR060311"
 			(at 0 0 0)
 			(hide yes)
@@
 			)
 		)
-		(property "MPN" "GPN"
+		(property "MPN" "GPR060310K"
 			(at 13.97 2.54 0)
 			(hide yes)
@@
 			)
 		)
-		(property "MPN" "GPN"
+		(property "MPN" "GPC1206106"
 			(at 0 0 0)
 			(hide yes)
@@
 			)
 		)
-		(property "MPN" "GPN"
+		(property "MPN" "GPC0603475"
 			(at 0 0 0)
 			(hide yes)
@@
 			)
 		)
-		(property "MPN" "GPN"
+		(property "MPN" "GPR0603301"
 			(at 0 0 0)
 			(hide yes)
@@
 			)
 		)
-		(property "MPN" "GPN"
+		(property "MPN" "GPC1206226"
 			(at 0 0 0)
 			(hide yes)
@@
 			)
 		)
-		(property "MPN" "GPN"
+		(property "MPN" "GPC0603473"
 			(at 0 0 0)
 			(hide yes)
@@
 			)
 		)
-		(property "MPN" "GPN"
+		(property "MPN" "GPR0603523"
 			(at 0 0 0)
 			(hide yes)
@@
 			)
 		)
-		(property "MPN" "GPN"
+		(property "MPN" "GPR0603300R"
 			(at 0 0 0)
 			(hide yes)
@@
 			)
 		)
-		(property "MPN" "GPN"
+		(property "MPN" "GPR060322"
 			(at 0 0 0)
 			(hide yes)
