File: recharger.kicad_sch (KiCad schematic)
At the start: 23 parts, among them J9 Battery Connector, U2 BQ25887RGE

Commit message: finalizing pcb
Parts:
- removed R21: 10k, Resistor_SMD:R_0603_1608Metric, symbol Device:R
- C12, C3: LCSC C77091 -> C53084537
- C7: LCSC C29519229 -> C86295
Connections:
- net GND: now also U2.24 (PSEL)
Changed lines of the file:
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@@
 	)
 	(junction
-		(at 99.06 101.6)
-		(diameter 0)
-		(color 0 0 0 0)
-	)
-	(junction
 		(at 158.75 121.92)
 		(diameter 0)
@@
 	)
 	(no_connect
-		(at 194.31 99.06)
+		(at 132.08 106.68)
 	)
 	(no_connect
-		(at 132.08 106.68)
+		(at 194.31 99.06)
 	)
 	(bus_entry
@@
 	(wire
 		(pts
-			(xy 93.98 101.6) (xy 99.06 101.6)
-		)
-		(stroke
-			(width 0)
-			(type default)
-		)
-	)
-	(wire
-		(pts
 			(xy 119.38 86.36) (xy 132.08 86.36)
 		)
@@
 	(wire
 		(pts
-			(xy 121.92 104.14) (xy 132.08 104.14)
+			(xy 176.53 99.06) (xy 176.53 104.14)
 		)
 		(stroke
@@
 	(wire
 		(pts
-			(xy 176.53 99.06) (xy 176.53 104.14)
+			(xy 163.83 106.68) (xy 173.99 106.68)
 		)
 		(stroke
@@
 	(wire
 		(pts
-			(xy 163.83 106.68) (xy 173.99 106.68)
+			(xy 127 116.84) (xy 127 118.11)
 		)
 		(stroke
@@
 	(wire
 		(pts
-			(xy 127 116.84) (xy 127 118.11)
+			(xy 158.75 120.65) (xy 158.75 121.92)
 		)
 		(stroke
@@
 	(wire
 		(pts
-			(xy 158.75 120.65) (xy 158.75 121.92)
+			(xy 132.08 104.14) (xy 127 104.14)
 		)
 		(stroke
@@
 		)
 	)
-	(wire
-		(pts
-			(xy 99.06 104.14) (xy 99.06 101.6)
-		)
-		(stroke
-			(width 0)
-			(type default)
-		)
-	)
 	(bus
 		(pts
@@
 	(wire
 		(pts
+			(xy 127 104.14) (xy 127 105.41)
+		)
+		(stroke
+			(width 0)
+			(type default)
+		)
+	)
+	(wire
+		(pts
 			(xy 116.84 125.73) (xy 116.84 127)
 		)
@@
 	(wire
 		(pts
-			(xy 99.06 101.6) (xy 100.33 101.6)
+			(xy 93.98 101.6) (xy 100.33 101.6)
 		)
 		(stroke
@@
 	(wire
 		(pts
-			(xy 114.3 104.14) (xy 99.06 104.14)
-		)
-		(stroke
-			(width 0)
-			(type default)
-		)
-	)
-	(wire
-		(pts
 			(xy 152.4 106.68) (xy 156.21 106.68)
 		)
@@
 			)
 		)
-		(property "LCSC" "C77091"
+		(property "LCSC" "C53084537"
 			(at 0 0 0)
 			(hide yes)
@@
 	)
 	(symbol
-		(lib_id "Device:C")
-		(at 207.01 86.36 0)
+		(lib_id "power:GND")
+		(at 127 105.41 0)
 		(unit 1)
 		(body_style 1)
@@
 		(dnp no)
 		(fields_autoplaced yes)
-		(property "Reference" "C7"
-			(at 210.82 85.0899 0)
-			(show_name no)
-			(do_not_autoplace no)
-			(effects
-				(font
-					(size 1.27 1.27)
-				)
-				(justify left)
-			)
-		)
-		(property "Value" "22uF"
-			(at 210.82 87.6299 0)
-			(show_name no)
-			(do_not_autoplace no)
-			(effects
-				(font
-					(size 1.27 1.27)
-				)
-				(justify left)
-			)
-		)
-		(property "Footprint" "Capacitor_SMD:C_0603_1608Metric"
-			(at 207.9752 90.17 0)
+		(property "Reference" "#PWR069"
+			(at 127 111.76 0)
 			(hide yes)
 			(show_name no)
@@
 			)
 		)
-		(property "Datasheet" "https://datasheet.lcsc.com/datasheet/pdf/02336ea48ea44ca18c72517dd3cb7b47.pdf?productCode=C962136"
-			(at 207.01 86.36 0)
-			(hide yes)
-			(show_name no)
-			(do_not_autoplace no)
-			(effects
-				(font
-					(size 1.27 1.27)
-				)
-			)
-		)
-		(property "Description" "Unpolarized capacitor"
-			(at 207.01 86.36 0)
-			(hide yes)
+		(property "Value" "GND"
+			(at 127 110.49 0)
 			(show_name no)
 			(do_not_autoplace no)
@@
 			)
 		)
-		(property "Manufacturer" "Murata"
-			(at 0 0 0)
+		(property "Footprint" ""
+			(at 127 105.41 0)
 			(hide yes)
 			(show_name no)
@@
 			)
 		)
-		(property "MPN" "GRM188C61E226ME01D"
-			(at 0 0 0)
+		(property "Datasheet" ""
+			(at 127 105.41 0)
 			(hide yes)
 			(show_name no)
@@
 			)
 		)
-		(property "LCSC" "C29519229"
-			(at 0 0 0)
+		(property "Description" "Power symbol creates a global label with name \"GND\" , ground"
+			(at 127 105.41 0)
 			(hide yes)
 			(show_name no)
@@
 		(pin "1"
 		)
-		(pin "2"
-		)
 		(instances
 			(project "rover-circuit"
 				(path "/0461baee-3b25-4e1a-a5c1-d76b4b99c66c/d12ae2b7-4c48-4e18-8e74-760d158fba59"
-					(reference "C7")
+					(reference "#PWR069")
 					(unit 1)
 				)
@@
 	)
 	(symbol
-		(lib_id "Device:R")
-		(at 127 121.92 0)
+		(lib_id "Device:C")
+		(at 207.01 86.36 0)
 		(unit 1)
 		(body_style 1)
@@
 		(dnp no)
 		(fields_autoplaced yes)
-		(property "Reference" "R2"
-			(at 129.54 120.6499 0)
+		(property "Reference" "C7"
+			(at 210.82 85.0899 0)
 			(show_name no)
 			(do_not_autoplace no)
@@
 			)
 		)
-		(property "Value" "1.1K"
-			(at 129.54 123.1899 0)
+		(property "Value" "22uF"
+			(at 210.82 87.6299 0)
 			(show_name no)
 			(do_not_autoplace no)
@@
 			)
 		)
-		(property "Footprint" "Resistor_SMD:R_0603_1608Metric"
-			(at 125.222 121.92 90)
+		(property "Footprint" "Capacitor_SMD:C_0603_1608Metric"
+			(at 207.9752 90.17 0)
 			(hide yes)
 			(show_name no)
@@
 			)
 		)
-		(property "Datasheet" "https://datasheet.lcsc.com/datasheet/pdf/0a975aaa49b7c97f38a963127be4a823.pdf?productCode=C22764"
-			(at 127 121.92 0)
+		(property "Datasheet" "https://datasheet.lcsc.com/datasheet/pdf/02336ea48ea44ca18c72517dd3cb7b47.pdf?productCode=C962136"
+			(at 207.01 86.36 0)
 			(hide yes)
 			(show_name no)
@@
 			)
 		)
-		(property "Description" "Resistor"
-			(at 127 121.92 0)
+		(property "Description" "Unpolarized capacitor"
+			(at 207.01 86.36 0)
 			(hide yes)
 			(show_name no)
@@
 			)
 		)
-		(property "Manufacturer" "Generic"
+		(property "Manufacturer" "Murata"
 			(at 0 0 0)
 			(hide yes)
@@
 			)
 		)
-		(property "MPN" "GPR060311"
+		(property "MPN" "GRM188C61E226ME01D"
 			(at 0 0 0)
 			(hide yes)
@@
 			)
 		)
-		(property "LCSC" "C22764"
+		(property "LCSC" "C86295"
 			(at 0 0 0)
 			(hide yes)
@@
 			)
 		)
-		(pin "2"
-		)
 		(pin "1"
 		)
+		(pin "2"
+		)
 		(instances
 			(project "rover-circuit"
 				(path "/0461baee-3b25-4e1a-a5c1-d76b4b99c66c/d12ae2b7-4c48-4e18-8e74-760d158fba59"
-					(reference "R2")
+					(reference "C7")
 					(unit 1)
 				)
@@
 	(symbol
 		(lib_id "Device:R")
-		(at 118.11 104.14 90)
+		(at 127 121.92 0)
 		(unit 1)
 		(body_style 1)
@@
 		(dnp no)
 		(fields_autoplaced yes)
-		(property "Reference" "R21"
-			(at 118.11 97.79 90)
+		(property "Reference" "R2"
+			(at 129.54 120.6499 0)
 			(show_name no)
 			(do_not_autoplace no)
@@
 					(size 1.27 1.27)
 				)
+				(justify left)
 			)
 		)
-		(property "Value" "10k"
-			(at 118.11 100.33 90)
+		(property "Value" "1.1K"
+			(at 129.54 123.1899 0)
 			(show_name no)
 			(do_not_autoplace no)
@@
 					(size 1.27 1.27)
 				)
+				(justify left)
 			)
 		)
 		(property "Footprint" "Resistor_SMD:R_0603_1608Metric"
-			(at 118.11 105.918 90)
+			(at 125.222 121.92 90)
 			(hide yes)
 			(show_name no)
@@
 			)
 		)
-		(property "Datasheet" "https://datasheet.lcsc.com/datasheet/pdf/b3641306390dfb6f98ec07837c926b58.pdf?productCode=C2906982"
-			(at 118.11 104.14 0)
+		(property "Datasheet" "https://datasheet.lcsc.com/datasheet/pdf/0a975aaa49b7c97f38a963127be4a823.pdf?productCode=C22764"
+			(at 127 121.92 0)
 			(hide yes)
 			(show_name no)
@@
 		)
 		(property "Description" "Resistor"
-			(at 118.11 104.14 0)
+			(at 127 121.92 0)
 			(hide yes)
 			(show_name no)
@@
 		)
 		(property "Manufacturer" "Generic"
-			(at 13.97 2.54 0)
+			(at 0 0 0)
 			(hide yes)
 			(show_name no)
@@
 			)
 		)
-		(property "MPN" "GPR060310K"
-			(at 13.97 2.54 0)
+		(property "MPN" "GPR060311"
+			(at 0 0 0)
 			(hide yes)
 			(show_name no)
@@
 			)
 		)
-		(property "LCSC" "C15401"
-			(at 13.97 2.54 0)
+		(property "LCSC" "C22764"
+			(at 0 0 0)
 			(hide yes)
 			(show_name no)
@@
 			)
 		)
-		(pin "1"
-		)
 		(pin "2"
 		)
+		(pin "1"
+		)
 		(instances
 			(project "rover-circuit"
 				(path "/0461baee-3b25-4e1a-a5c1-d76b4b99c66c/d12ae2b7-4c48-4e18-8e74-760d158fba59"
-					(reference "R21")
+					(reference "R2")
 					(unit 1)
 				)
@@
 			)
 		)
-		(property "LCSC" "C77091"
+		(property "LCSC" "C53084537"
 			(at 0 0 0)
 			(hide yes)
