File: imu.kicad_sch (KiCad schematic)
At the start: 6 parts, among them U1 MMC5983MA, U11 BMI270

Commit message: add MPS entries
Parts:
- C14, C15: MPN CL10A106KO8NQNC -> GPN; Manufacturer Samsung Electro-Mechanics -> Generic
- C29, C30: MPN CC0603KRX7R9BB104 -> GPN; Manufacturer YAGEO -> Generic
Changed lines of the file:
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@@
 			)
 		)
-		(property "Manufacturer" "Samsung Electro-Mechanics"
-			(at 0 0 0)
-			(hide yes)
-			(show_name no)
-			(do_not_autoplace no)
-			(effects
-				(font
-					(size 1.27 1.27)
-				)
-			)
-		)
-		(property "MPN" "CL10A106KO8NQNC"
+		(property "Manufacturer" "Generic"
+			(at 0 0 0)
+			(hide yes)
+			(show_name no)
+			(do_not_autoplace no)
+			(effects
+				(font
+					(size 1.27 1.27)
+				)
+			)
+		)
+		(property "MPN" "GPN"
 			(at 0 0 0)
 			(hide yes)
@@
 			)
 		)
-		(property "Manufacturer" "Samsung Electro-Mechanics"
-			(at 0 0 0)
-			(hide yes)
-			(show_name no)
-			(do_not_autoplace no)
-			(effects
-				(font
-					(size 1.27 1.27)
-				)
-			)
-		)
-		(property "MPN" "CL10A106KO8NQNC"
+		(property "Manufacturer" "Generic"
+			(at 0 0 0)
+			(hide yes)
+			(show_name no)
+			(do_not_autoplace no)
+			(effects
+				(font
+					(size 1.27 1.27)
+				)
+			)
+		)
+		(property "MPN" "GPN"
 			(at 0 0 0)
 			(hide yes)
@@
 			)
 		)
-		(property "Manufacturer" "YAGEO"
-			(at 0 0 0)
-			(hide yes)
-			(show_name no)
-			(do_not_autoplace no)
-			(effects
-				(font
-					(size 1.27 1.27)
-				)
-			)
-		)
-		(property "MPN" "CC0603KRX7R9BB104"
+		(property "Manufacturer" "Generic"
+			(at 0 0 0)
+			(hide yes)
+			(show_name no)
+			(do_not_autoplace no)
+			(effects
+				(font
+					(size 1.27 1.27)
+				)
+			)
+		)
+		(property "MPN" "GPN"
 			(at 0 0 0)
 			(hide yes)
@@
 			)
 		)
-		(property "Manufacturer" "YAGEO"
-			(at 0 0 0)
-			(hide yes)
-			(show_name no)
-			(do_not_autoplace no)
-			(effects
-				(font
-					(size 1.27 1.27)
-				)
-			)
-		)
-		(property "MPN" "CC0603KRX7R9BB104"
-			(at 0 0 0)
-			(hide yes)
+		(property "Manufacturer" "Generic"
+			(at 0 0 0)
+			(hide yes)
+			(show_name no)
+			(do_not_autoplace no)
+			(effects
+				(font
+					(size 1.27 1.27)
+				)
+			)
+		)
+		(property "MPN" "GPN"
+			(at 0 0 0)
+			(hide yes)

Commit message: update MPN codes
Parts:
- C14, C15: MPN GPN -> GPC0603106
- C29, C30: MPN GPN -> GPC0603104
Changed lines of the file:
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@@
 			)
 		)
-		(property "MPN" "GPN"
+		(property "MPN" "GPC0603106"
 			(at 0 0 0)
 			(hide yes)
@@
 			)
 		)
-		(property "MPN" "GPN"
+		(property "MPN" "GPC0603106"
 			(at 0 0 0)
 			(hide yes)
@@
 			)
 		)
-		(property "MPN" "GPN"
+		(property "MPN" "GPC0603104"
 			(at 0 0 0)
 			(hide yes)
@@
 			)
 		)
-		(property "MPN" "GPN"
-			(at 0 0 0)
-			(hide yes)
+		(property "MPN" "GPC0603104"
+			(at 0 0 0)
+			(hide yes)
