File: mcu.kicad_sch (KiCad schematic)
At the start: 4 parts, among them SW1 SW_EN, SW2 SW_IO0, U6 ESP32-C6-WROOM-1-N8

Commit message: tentative automatic population
Parts:
- C1: LCSC C60474 -> C49678; MPN (none) -> CC0805KRX7R9BB104; Manufacturer (none) -> YAGEO
- SW1, SW2: MPN (none) -> B3U-1000P; Manufacturer (none) -> OMRON
- U6: LCSC (none) -> C5366877; MPN (none) -> ESP32-C6-WROOM-1-N8; Manufacturer (none) -> ESPRESSIF
Changed lines of the file:
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@@
 			)
 		)
-		(property "Datasheet" ""
+		(property "Datasheet" "https://datasheet.lcsc.com/datasheet/pdf/23ccee80ee542e7cf156a772bb589942.pdf?productCode=C49678"
 			(at 138.43 46.99 0)
 			(hide yes)
@@
 			)
 		)
-		(property "LCSC" "C60474"
+		(property "LCSC" "C49678"
 			(at 138.43 46.99 0)
 			(hide yes)
@@
 					(size 1.27 1.27)
 				)
+			)
+		)
+		(property "Manufacturer" "YAGEO" (at 0 0 0)
+			(effects
+				(font
+					(size 1.27 1.27)
+				)
+				(hide yes)
+			)
+		)
+		(property "MPN" "CC0805KRX7R9BB104" (at 0 0 0)
+			(effects
+				(font
+					(size 1.27 1.27)
+				)
+				(hide yes)
 			)
 		)
@@
 			)
 		)
-		(property "Datasheet" ""
+		(property "Datasheet" "https://datasheet.lcsc.com/datasheet/pdf/5613ec928e7c35b77f993ac0df056a32.pdf?productCode=C231329"
 			(at 125.73 146.05 0)
 			(hide yes)
@@
 					(size 1.27 1.27)
 				)
+			)
+		)
+		(property "Manufacturer" "OMRON" (at 0 0 0)
+			(effects
+				(font
+					(size 1.27 1.27)
+				)
+				(hide yes)
+			)
+		)
+		(property "MPN" "B3U-1000P" (at 0 0 0)
+			(effects
+				(font
+					(size 1.27 1.27)
+				)
+				(hide yes)
 			)
 		)
@@
 			)
 		)
-		(property "Datasheet" ""
+		(property "Datasheet" "https://datasheet.lcsc.com/datasheet/pdf/914ba3f9643762e2fb21b3ff300ff859.pdf?productCode=C5366877"
 			(at 138.43 90.17 0)
 			(hide yes)
@@
 				)
 				(justify bottom)
+			)
+		)
+		(property "MPN" "ESP32-C6-WROOM-1-N8" (at 0 0 0)
+			(effects
+				(font
+					(size 1.27 1.27)
+				)
+				(hide yes)
+			)
+		)
+		(property "Manufacturer" "ESPRESSIF" (at 0 0 0)
+			(effects
+				(font
+					(size 1.27 1.27)
+				)
+				(hide yes)
+			)
+		)
+		(property "LCSC" "C5366877" (at 0 0 0)
+			(effects
+				(font
+					(size 1.27 1.27)
+				)
+				(hide yes)
 			)
 		)
@@
 			)
 		)
-		(property "Datasheet" ""
+		(property "Datasheet" "https://datasheet.lcsc.com/datasheet/pdf/5613ec928e7c35b77f993ac0df056a32.pdf?productCode=C231329"
 			(at 142.24 146.05 0)
 			(hide yes)
@@
 			)
 		)
+		(property "Manufacturer" "OMRON" (at 0 0 0)
+			(effects
+				(font
+					(size 1.27 1.27)
+				)
+				(hide yes)
+			)
+		)
+		(property "MPN" "B3U-1000P" (at 0 0 0)
+			(effects
+				(font
+					(size 1.27 1.27)
+				)
+				(hide yes)
+			)
+		)

Commit message: Consistent final layout
Connections:
- net ~{INT}: now also U6.19 (IO21); no longer U6.18 (IO20)
- net ~{KILL}: now also U6.18 (IO20); no longer U6.19 (IO21)
Changed lines of the file:
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@@
 	(hierarchical_label "~{KILL}"
 		(shape output)
-		(at 163.83 100.33 0)
+		(at 163.83 97.79 0)
 		(effects
 			(font
@@
 	(hierarchical_label "~{INT}"
 		(shape input)
-		(at 163.83 97.79 0)
+		(at 163.83 100.33 0)
 		(effects
 			(font
@@
 			)
 		)
-		(property "Manufacturer" "YAGEO" (at 0 0 0)
-			(effects
-				(font
-					(size 1.27 1.27)
-				)
-				(hide yes)
-			)
-		)
-		(property "MPN" "CC0805KRX7R9BB104" (at 0 0 0)
-			(effects
-				(font
-					(size 1.27 1.27)
-				)
-				(hide yes)
+		(property "Manufacturer" "YAGEO"
+			(at 0 0 0)
+			(hide yes)
+			(show_name no)
+			(do_not_autoplace no)
+			(effects
+				(font
+					(size 1.27 1.27)
+				)
+			)
+		)
+		(property "MPN" "CC0805KRX7R9BB104"
+			(at 0 0 0)
+			(hide yes)
+			(show_name no)
+			(do_not_autoplace no)
+			(effects
+				(font
+					(size 1.27 1.27)
+				)
 			)
 		)
@@
 			)
 		)
-		(property "Manufacturer" "OMRON" (at 0 0 0)
-			(effects
-				(font
-					(size 1.27 1.27)
-				)
-				(hide yes)
-			)
-		)
-		(property "MPN" "B3U-1000P" (at 0 0 0)
-			(effects
-				(font
-					(size 1.27 1.27)
-				)
-				(hide yes)
+		(property "Manufacturer" "OMRON"
+			(at 0 0 0)
+			(hide yes)
+			(show_name no)
+			(do_not_autoplace no)
+			(effects
+				(font
+					(size 1.27 1.27)
+				)
+			)
+		)
+		(property "MPN" "B3U-1000P"
+			(at 0 0 0)
+			(hide yes)
+			(show_name no)
+			(do_not_autoplace no)
+			(effects
+				(font
+					(size 1.27 1.27)
+				)
 			)
 		)
@@
 			)
 		)
-		(property "MPN" "ESP32-C6-WROOM-1-N8" (at 0 0 0)
-			(effects
-				(font
-					(size 1.27 1.27)
-				)
-				(hide yes)
-			)
-		)
-		(property "Manufacturer" "ESPRESSIF" (at 0 0 0)
-			(effects
-				(font
-					(size 1.27 1.27)
-				)
-				(hide yes)
-			)
-		)
-		(property "LCSC" "C5366877" (at 0 0 0)
-			(effects
-				(font
-					(size 1.27 1.27)
-				)
-				(hide yes)
+		(property "MPN" "ESP32-C6-WROOM-1-N8"
+			(at 0 0 0)
+			(hide yes)
+			(show_name no)
+			(do_not_autoplace no)
+			(effects
+				(font
+					(size 1.27 1.27)
+				)
+			)
+		)
+		(property "Manufacturer" "ESPRESSIF"
+			(at 0 0 0)
+			(hide yes)
+			(show_name no)
+			(do_not_autoplace no)
+			(effects
+				(font
+					(size 1.27 1.27)
+				)
+			)
+		)
+		(property "LCSC" "C5366877"
+			(at 0 0 0)
+			(hide yes)
+			(show_name no)
+			(do_not_autoplace no)
+			(effects
+				(font
+					(size 1.27 1.27)
+				)
 			)
 		)
@@
 			)
 		)
-		(property "Manufacturer" "OMRON" (at 0 0 0)
-			(effects
-				(font
-					(size 1.27 1.27)
-				)
-				(hide yes)
-			)
-		)
-		(property "MPN" "B3U-1000P" (at 0 0 0)
-			(effects
-				(font
-					(size 1.27 1.27)
-				)
-				(hide yes)
-			)
-		)
+		(property "Manufacturer" "OMRON"
+			(at 0 0 0)
+			(hide yes)
+			(show_name no)
+			(do_not_autoplace no)
+			(effects
+				(font
+					(size 1.27 1.27)
+				)
+			)
+		)
+		(property "MPN" "B3U-1000P"
+			(at 0 0 0)
+			(hide yes)
+			(show_name no)
+			(do_not_autoplace no)
+			(effects
+				(font
+					(size 1.27 1.27)
+				)
+			)
+		)

Commit message: finalized component selection
Parts:
- C1: value 100n -> 100nF 0805 X7R MLCC
Changed lines of the file:
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@@
 	)
 	(bus_entry
-		(at 102.87 92.71)
+		(at 100.33 92.71)
 		(size 2.54 2.54)
 		(stroke
@@
 	)
 	(bus_entry
-		(at 102.87 87.63)
+		(at 100.33 87.63)
 		(size 2.54 2.54)
 		(stroke
@@
 	)
 	(bus_entry
-		(at 102.87 90.17)
+		(at 100.33 90.17)
 		(size 2.54 2.54)
 		(stroke
@@
 	(bus
 		(pts
-			(xy 102.87 85.09) (xy 102.87 92.71)
+			(xy 100.33 85.09) (xy 100.33 92.71)
 		)
 		(stroke
@@
 	(bus
 		(pts
-			(xy 101.6 83.82) (xy 102.87 85.09)
+			(xy 99.06 83.82) (xy 100.33 85.09)
 		)
 		(stroke
@@
 	(wire
 		(pts
-			(xy 105.41 95.25) (xy 120.65 95.25)
+			(xy 102.87 95.25) (xy 120.65 95.25)
 		)
 		(stroke
@@
 	(wire
 		(pts
-			(xy 105.41 90.17) (xy 120.65 90.17)
+			(xy 102.87 90.17) (xy 120.65 90.17)
 		)
 		(stroke
@@
 	(wire
 		(pts
-			(xy 105.41 92.71) (xy 120.65 92.71)
+			(xy 102.87 92.71) (xy 120.65 92.71)
 		)
 		(stroke
@@
 	(bus
 		(pts
-			(xy 97.79 83.82) (xy 101.6 83.82)
+			(xy 95.25 83.82) (xy 99.06 83.82)
 		)
 		(stroke
@@
 	(hierarchical_label "{MISO MOSI CLK}"
 		(shape bidirectional)
-		(at 97.79 83.82 180)
+		(at 95.25 83.82 180)
 		(effects
 			(font
@@
 			)
 		)
-		(property "Value" "100n"
+		(property "Value" "100nF 0805 X7R MLCC"
 			(at 142.24 48.2599 0)
 			(show_name no)

Commit message: add MPS entries
Parts:
- C1: MPN CC0805KRX7R9BB104 -> GPN; Manufacturer YAGEO -> Generic
Changed lines of the file:
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@@
 			)
 		)
-		(property "Manufacturer" "YAGEO"
+		(property "Manufacturer" "Generic"
 			(at 0 0 0)
 			(hide yes)
@@
 			)
 		)
-		(property "MPN" "CC0805KRX7R9BB104"
+		(property "MPN" "GPN"
 			(at 0 0 0)
 			(hide yes)

Commit message: update MPN codes
Parts:
- C1: MPN GPN -> GPC0805104
Changed lines of the file:
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@@
 			)
 		)
-		(property "MPN" "GPN"
+		(property "MPN" "GPC0805104"
 			(at 0 0 0)
 			(hide yes)
