File: mcu.kicad_sch (KiCad schematic)
At the start: 4 parts, among them SW1 SW_EN, SW2 SW_IO0, U6 ESP32-C6-WROOM-1-N8

Commit message: finalizing pcb
Parts:
- C1: LCSC C49678 -> C326595
Changed lines of the file:
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@@
 			)
 		)
-		(property "LCSC" "C49678"
+		(property "LCSC" "C326595"
 			(at 138.43 46.99 0)
 			(hide yes)

Commit message: solve a problem with enable resistor and capacitor
Parts:
- added C33: 0.1uF, Capacitor_SMD:C_0805_2012Metric, symbol Device:C
- added R21: 10k, Resistor_SMD:R_0603_1608Metric, symbol Device:R
Connections:
- net +3V3: now also R21.1
- net EN: now also C33.2, R21.2
- net GND: now also C33.1

Commit message: finalizing minor issues and improvements
Parts:
- C1: value 100nF 0805 X7R MLCC -> 0.1uF; LCSC C326595 -> C49678; MPN GPC0805104 -> (none)
Changed lines of the file:
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@@
 			)
 		)
-		(property "Value" "100nF 0805 X7R MLCC"
+		(property "Value" "0.1uF"
 			(at 142.24 48.2599 0)
 			(show_name no)
@@
 			)
 		)
-		(property "LCSC" "C326595"
+		(property "LCSC" "C49678"
 			(at 138.43 46.99 0)
 			(hide yes)
@@
 			)
 		)
-		(property "MPN" "GPC0805104"
+		(property "MPN" ""
 			(at 0 0 0)
 			(hide yes)
