File: usb.kicad_sch (KiCad schematic)
At the start: 5 parts, among them J2 USB C Connector, U4 TPD2EUSB30

Commit message: finalizing minor issues and improvements
Parts:
- added C35: 1uF, Capacitor_SMD:C_0603_1608Metric, symbol Device:C
Connections:
- net GND: now also C35.2
- net VBUS: now also C35.1
