File: sbc.kicad_sch (KiCad schematic)
At the start: 2 parts, among them J5 Raspberry Pi Hat Connector, J6 Expansion Header

Commit message: add proper labels and minors improvements
Connections:
- net IO12: now reaches J6.10 (Pin_10)
- net IO12: now also J5.32 (PWM0/GPIO12)
- no-connect marks 26 -> 24
Changed lines of the file:
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@@
-	)
-	(no_connect
-		(at 142.24 111.76)
 	)
 	(no_connect
@@
 	(no_connect
 		(at 101.6 99.06)
-	)
-	(no_connect
-		(at 193.04 97.79)
 	)
 	(no_connect
@@
 	(wire
 		(pts
+			(xy 142.24 111.76) (xy 147.32 111.76)
+		)
+		(stroke
+			(width 0)
+			(type default)
+		)
+	)
+	(wire
+		(pts
 			(xy 157.48 81.28) (xy 157.48 95.25)
 		)
@@
 		(pts
 			(xy 160.02 92.71) (xy 180.34 92.71)
+		)
+		(stroke
+			(width 0)
+			(type default)
+		)
+	)
+	(wire
+		(pts
+			(xy 193.04 97.79) (xy 207.01 97.79)
 		)
 		(stroke
@@
 		)
 	)
+	(label "IO12"
+		(at 147.32 111.76 0)
+		(effects
+			(font
+				(size 1.27 1.27)
+			)
+			(justify left bottom)
+		)
+	)
 	(label "SDA"
 		(at 198.12 100.33 0)
 		(effects
 			(font
+				(size 1.27 1.27)
+			)
+			(justify left bottom)
+		)
+	)
+	(label "IO12"
+		(at 207.01 97.79 0)
+		(effects
+			(font
